File: ECU-Designs/Cooling-ECU/Cooling1.brd (EAGLE design)
At the start: 100 x 80 mm, 11 parts

Commit message: Cooling board update and file cleanup
Parts:
- added U$3, U$4, U$5: PSMN011_MOSFET, HyTechDevices:SOT669
- moved R4 9.25 mm to (41.9, 36.8)
- moved R2 6.48 mm to (50.8, 49.5)
- moved R3 6.48 mm to (50.8, 47.0)
- moved R1 1.27 mm to (26.7, 26.7)
Connections:
- net 12V_COOLING_SUPPLY: now also U$3.MB, U$3.MB2, U$4.MB, U$4.MB2, U$5.MB, U$5.MB2
- net GND: now also U$3.1, U$3.2, U$3.3, U$4.1, U$4.2, U$4.3, U$5.1, U$5.2, U$5.3
- net N$17: now also U$4.4
- net N$4: now also U$5.4
- net N$6: now also U$3.4
Routing:
- net 12V_COOLING_SUPPLY: track 59.7 -> 123.5 mm
- net 5V: track 20.3 -> 58.3 mm
- net GND: track 44.7 -> 74.0 mm, vias 0 -> 1
- net N$6: track 0.00 -> 12.4 mm
- net N$1: track 4.82 -> 13.1 mm
- net N$4: track 0.00 -> 5.90 mm
- net N$9: track 5.98 -> 1.64 mm
- net N$12: track 5.98 -> 1.64 mm
- net N$17: track 19.6 -> 23.9 mm, vias 0 -> 2
- net N$8: track 20.9 -> 18.9 mm
- added copper zone on layer 1, net GND
- added copper zone on layer 16, net GND
Other:
- board size 100 x 80 mm -> 42.9 x 43.2 mm
