File: ECU-Designs/Cooling-ECU/Cooling_flowSensor.brd (EAGLE design)
At the start: 42.9 x 43.2 mm, 16 parts

Commit message: Updated cooling board
Parts:
- removed 12V_COOLING_SUPPLY: MINIFIT_5566-2, HyTechDevices:MINIFIT_5566-2
- removed FAN/PUMP: MINIFIT_5566-4, HyTechDevices:MINIFIT_5566-4
- added X1: MINIFIT_5566-6, HyTechDevices:MINIFIT_5566-6
- added X2: MINIFIT_5566-4, HyTechDevices:MINIFIT_5566-4
- moved U$4 35.3 mm to (38.1, 58.4), turned to 0 degrees
- moved R1 22.9 mm to (19.1, 48.3)
- moved OUT 21.7 mm to (19.1, 48.3)
- moved R4 21.1 mm to (30.5, 54.6), turned to 270 degrees
- moved FLOW_SENSOR 19.7 mm to (50.8, 34.3), turned to 270 degrees
- moved U$5 15.3 mm to (31.8, 61.0)
- moved R5 14.5 mm to (45.7, 44.5), turned to 270 degrees
- moved IC1 13.7 mm to (19.1, 61.0)
- moved R3 13.7 mm to (38.1, 52.1), turned to 180 degrees
- moved IN 9.16 mm to (19.1, 35.6)
- moved U$1 8.98 mm to (25.4, 29.2)
- moved U$3 8.03 mm to (34.3, 34.3), turned to 180 degrees
- moved R2 6.48 mm to (45.7, 52.1), turned to 270 degrees
- moved U$2 6.35 mm to (30.5, 45.7)
Connections:
- net N$11 renamed CAN-H
- net N$8 renamed CAN-L
- removed net 12V_COOLING_SUPPLY: 12V_COOLING_SUPPLY.1, FAN/PUMP.1, FAN/PUMP.2, FAN/PUMP.3, U$3.MB, U$3.MB2, U$4.MB, U$4.MB2, U$5.MB, U$5.MB2
- removed net N$4 (its old number): R2.2, U$5.4
- removed net N$6 (its old number): R4.1, U$3.4
- new net AUX_12V_1: X1.1, X2.1
- new net AUX_12V_2: X1.3
- new net AUX_12V_3: X1.5, X2.3
- new net N$13: R4.1, U$5.4
- new net N$14: U$4.MB, U$4.MB2, X1.4
- new net N$15: U$5.MB, U$5.MB2, X1.6
- new net N$19: U$3.MB, U$3.MB2, X1.2
- new net N$9: R2.2, U$3.4
- net GND: now also U$2.8
Routing:
- net 12V_COOLING_SUPPLY: track 132.6 -> 0.00 mm, vias 3 -> 0
- net N$19: track 0.00 -> 53.9 mm, vias 0 -> 2
- net N$15: track 0.00 -> 38.5 mm
- net N$14: track 0.00 -> 31.9 mm
- net 12V: track 99.6 -> 70.4 mm
- net GND: track 50.0 -> 75.8 mm, vias 2 -> 5
- net N$9: track 0.00 -> 23.7 mm
- net AUX_12V_3: track 0.00 -> 22.9 mm
- net AUX_12V_1: track 0.00 -> 19.3 mm
- net N$12: track 23.9 -> 5.90 mm, vias 2 -> 0
- net N$7: track 2.82 -> 20.1 mm
- net N$10: track 19.4 -> 6.72 mm
- net N$6 (its old number): track 12.4 -> 0.00 mm
- net N$2: track 5.08 -> 16.5 mm
- net CAN-H: track 27.6 -> 34.4 mm
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Other:
- board size 42.9 x 43.2 mm -> 49.2 x 47 mm

Commit message: updated cooling board
Routing:
- net GND: track 75.8 -> 67.8 mm
- net 5V: track 65.1 -> 67.3 mm
Changed lines of the file:
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@@
 <grid distance="0.05" unitdist="inch" unit="inch" style="lines" multiple="1" display="no" altdistance="0.025" altunitdist="inch" altunit="inch"/>
 <layers>
-<layer number="1" name="Top" color="4" fill="1" visible="no" active="yes"/>
+<layer number="1" name="Top" color="4" fill="1" visible="yes" active="yes"/>
 <layer number="16" name="Bottom" color="1" fill="1" visible="yes" active="yes"/>
 <layer number="17" name="Pads" color="2" fill="1" visible="yes" active="yes"/>
@@
 </polygon>
 <wire x1="26.67" y1="63.5" x2="24.13" y2="63.5" width="0.6096" layer="16"/>
-<wire x1="27.94" y1="43.18" x2="27.94" y2="46.99" width="0.6096" layer="1"/>
 <wire x1="32.385" y1="37.015" x2="30.48" y2="37.015" width="0.6096" layer="16"/>
 <wire x1="30.48" y1="37.015" x2="30.48" y2="33.02" width="0.6096" layer="16"/>
 <via x="30.48" y="33.02" extent="1-16" drill="0.6" shape="square"/>
-<wire x1="30.48" y1="33.02" x2="29.21" y2="30.48" width="0.6096" layer="1"/>
 <wire x1="34.925" y1="37.015" x2="33.655" y2="37.015" width="0.6096" layer="16"/>
 <wire x1="33.655" y1="37.015" x2="32.385" y2="37.015" width="0.6096" layer="16"/>
 <wire x1="31.75" y1="45.72" x2="31.75" y2="48.26" width="0.6096" layer="16"/>
 <via x="31.75" y="48.26" extent="1-16" drill="0.6" shape="square"/>
-<wire x1="31.75" y1="48.26" x2="27.94" y2="48.26" width="0.6096" layer="1"/>
-<wire x1="27.94" y1="48.26" x2="27.94" y2="46.99" width="0.6096" layer="1"/>
-<wire x1="27.94" y1="46.99" x2="29.21" y2="46.99" width="0.6096" layer="1"/>
-<wire x1="29.21" y1="46.99" x2="29.21" y2="41.91" width="0.6096" layer="1"/>
-<wire x1="29.21" y1="41.91" x2="29.21" y2="36.83" width="0.6096" layer="1"/>
 <wire x1="30.48" y1="40.32" x2="29.21" y2="40.32" width="0.6096" layer="16"/>
-<wire x1="29.21" y1="40.32" x2="29.21" y2="41.91" width="0.6096" layer="16"/>
-<via x="29.21" y="41.91" extent="1-16" drill="0.6" shape="square"/>
+<wire x1="29.21" y1="40.32" x2="29.21" y2="43.18" width="0.6096" layer="16"/>
+<via x="29.21" y="43.18" extent="1-16" drill="0.6" shape="square"/>
 <wire x1="24.13" y1="63.5" x2="24.13" y2="57.15" width="0.6096" layer="16"/>
 <wire x1="24.13" y1="57.15" x2="21.3614" y2="57.15" width="0.6096" layer="16"/>
 <wire x1="21.3614" y1="57.15" x2="21.3614" y2="57.8612" width="0.6096" layer="16"/>
-<wire x1="34.29" y1="54.61" x2="33.02" y2="46.99" width="0.6096" layer="1"/>
-<wire x1="33.02" y1="46.99" x2="29.21" y2="46.99" width="0.6096" layer="1"/>
 <wire x1="31.115" y1="58.235" x2="32.385" y2="58.235" width="0.6096" layer="16"/>
 <wire x1="32.385" y1="58.235" x2="33.655" y2="58.235" width="0.6096" layer="16"/>
@@
 <wire x1="38.1" y1="54.61" x2="38.735" y2="54.61" width="0.6096" layer="16"/>
 <wire x1="38.735" y1="54.61" x2="38.735" y2="55.695" width="0.6096" layer="16"/>
+<wire x1="30.48" y1="33.02" x2="29.21" y2="33.02" width="0.6096" layer="1"/>
+<wire x1="29.21" y1="33.02" x2="29.21" y2="43.18" width="0.6096" layer="1"/>
+<wire x1="21.3614" y1="57.15" x2="21.15" y2="57.15" width="0.6096" layer="16"/>
+<wire x1="21.15" y1="57.15" x2="21.15" y2="51.01" width="0.6096" layer="16"/>
+<wire x1="29.21" y1="43.18" x2="29.21" y2="48.26" width="0.6096" layer="1"/>
+<wire x1="29.21" y1="48.26" x2="31.75" y2="48.26" width="0.6096" layer="1"/>
 <wire x1="38.735" y1="55.695" x2="40.005" y2="55.695" width="0" layer="19" extent="16-16"/>
 </signal>
@@
 <contactref element="IC1" pad="4"/>
 <wire x1="19.05" y1="64.059" x2="19.05" y2="67.31" width="0.6096" layer="16"/>
-<wire x1="19.05" y1="67.31" x2="43.18" y2="67.31" width="0.6096" layer="1"/>
-<wire x1="43.18" y1="67.31" x2="44.45" y2="63.5" width="0.6096" layer="1"/>
+<wire x1="19.05" y1="67.31" x2="44.45" y2="67.31" width="0.6096" layer="1"/>
+<wire x1="44.45" y1="67.31" x2="44.45" y2="63.5" width="0.6096" layer="1"/>
 <via x="19.05" y="67.31" extent="1-16" drill="0.6" shape="square"/>
 <wire x1="41.91" y1="63.5" x2="44.45" y2="63.5" width="0.6096" layer="16"/>
@@
 <wire x1="19.05" y1="57.8612" x2="19.05" y2="54.61" width="0.6096" layer="16"/>
 <via x="19.05" y="54.61" extent="1-16" drill="0.6" shape="square"/>
-<wire x1="19.05" y1="54.61" x2="31.75" y2="54.61" width="0.6096" layer="1"/>
-<wire x1="31.75" y1="54.61" x2="33.02" y2="48.26" width="0.6096" layer="1"/>
+<wire x1="19.05" y1="54.61" x2="33.02" y2="54.61" width="0.6096" layer="1"/>
+<wire x1="33.02" y1="54.61" x2="33.02" y2="48.26" width="0.6096" layer="1"/>
 <via x="33.02" y="48.26" extent="1-16" drill="0.6" shape="square"/>
 <wire x1="19.05" y1="64.059" x2="19.05" y2="57.8612" width="0.6096" layer="16"/>
@@
 <wire x1="39.37" y1="33.84" x2="39.37" y2="33.02" width="1.016" layer="16"/>
 <via x="39.37" y="33.02" extent="1-16" drill="0.6" shape="square"/>
-<wire x1="39.37" y1="33.02" x2="38.1" y2="27.94" width="1.016" layer="1"/>
-<wire x1="38.1" y1="27.94" x2="44.45" y2="27.94" width="1.016" layer="1"/>
-<wire x1="44.45" y1="27.94" x2="45.72" y2="59.69" width="1.016" layer="1"/>
-<wire x1="45.72" y1="59.69" x2="48.05" y2="59.69" width="1.016" layer="16"/>
-<via x="45.72" y="59.69" extent="1-16" drill="0.6" shape="square"/>
+<wire x1="39.37" y1="33.02" x2="39.37" y2="27.94" width="1.016" layer="1"/>
+<wire x1="39.37" y1="27.94" x2="44.45" y2="27.94" width="1.016" layer="1"/>
+<wire x1="44.45" y1="27.94" x2="44.45" y2="59.69" width="1.016" layer="1"/>
+<wire x1="44.45" y1="59.69" x2="48.05" y2="59.69" width="1.016" layer="16"/>
+<via x="44.45" y="59.69" extent="1-16" drill="0.6" shape="square"/>
 <wire x1="34.29" y1="33.84" x2="34.29" y2="31.54" width="0.6096" layer="16"/>
 </signal>
