File: ECU-Designs/Test Boards/BSPD Test Board.brd (EAGLE design)
At the start: 50.8 x 61.1 mm, 19 parts

Commit message: Tweak BSPD test board
Parts:
- C1: device HyTechDevices:0805 -> HyTechDevices:CAP-PTH-SMALLEZ
- R5: device HyTechDevices:0805 -> HyTechDevices:AXIAL-0.3EZ
- moved C1 3.54 mm to (33.8, 43.4)
- moved R3 3.30 mm to (33.8, 39.9)
- moved R5 2.84 mm to (37.3, 43.9)
Connections:
- net 5VSUPPLY: now also R5.P$2; no longer R5.2
- net N$13: now also R5.P$1; no longer R5.1
Routing:
- net N$13: track 74.1 -> 81.0 mm
- net N$14: track 54.5 -> 57.2 mm
- net GND: track 206.8 -> 205.5 mm
- net 5VSUPPLY: track 122.1 -> 122.6 mm
Other:
- board size 50.8 x 61.1 mm -> 50.8 x 57.3 mm
Changed lines of the file:
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@@
 <?xml version="1.0" encoding="utf-8"?>
 <!DOCTYPE eagle SYSTEM "eagle.dtd">
-<eagle version="7.6.0">
+<eagle version="7.7.0">
 <drawing>
 <settings>
@@
 <plain>
 <wire x1="0" y1="0" x2="50.78" y2="0" width="0" layer="20"/>
-<wire x1="50.78" y1="0" x2="50.78" y2="61.138" width="0" layer="20"/>
-<wire x1="50.78" y1="61.138" x2="0" y2="61.138" width="0" layer="20"/>
-<wire x1="0" y1="61.138" x2="0" y2="0" width="0" layer="20"/>
-<hole x="2.54" y="58.42" drill="3.2"/>
-<hole x="48.26" y="58.42" drill="3.2"/>
-<hole x="2.54" y="2.54" drill="3.2"/>
-<hole x="48.26" y="2.54" drill="3.2"/>
+<wire x1="50.78" y1="0" x2="50.78" y2="57.328" width="0" layer="20"/>
+<wire x1="50.78" y1="57.328" x2="0" y2="57.328" width="0" layer="20"/>
+<wire x1="0" y1="57.328" x2="0" y2="0" width="0" layer="20"/>
+<hole x="2.794" y="54.356" drill="3.2"/>
+<hole x="48.006" y="54.356" drill="3.2"/>
+<hole x="2.794" y="2.794" drill="3.2"/>
+<hole x="48.006" y="2.794" drill="3.2"/>
 </plain>
 <attributes>
@@
 <element name="AIR" library="HyTechDevices" package="LED-5MM" value="" x="25.4" y="31.75" rot="R180"/>
 <element name="BRAKE" library="HyTechDevices" package="TRIMPOT_3296" value="" x="17.78" y="25.4" rot="R90"/>
-<element name="C1" library="HyTechDevices" package="0805" value=".47u" x="35.052" y="46.736" rot="MR90"/>
+<element name="C1" library="HyTechDevices" package="CAP-PTH-SMALLEZ" value=".47u" x="33.782" y="43.434" rot="MR90"/>
 <element name="CALIBRATE1" library="HyTechDevices" package="TRIMPOT_3296" value="" x="11.43" y="52.07"/>
 <element name="CALIBRATE2" library="HyTechDevices" package="TRIMPOT_3296" value="" x="25.4" y="52.07"/>
@@
 <element name="R1" library="HyTechDevices" package="0805" value="" x="20.828" y="24.13" rot="MR0"/>
 <element name="R2" library="HyTechDevices" package="0805" value="" x="24.892" y="35.052" rot="MR180"/>
-<element name="R3" library="HyTechDevices" package="0805" value="330" x="35.052" y="42.926" rot="MR90"/>
+<element name="R3" library="HyTechDevices" package="0805" value="330" x="33.782" y="39.878" rot="MR90"/>
 <element name="R4" library="HyTechDevices" package="0805" value="" x="28.448" y="35.052" rot="MR180"/>
-<element name="R5" library="HyTechDevices" package="0805" value="430k" x="37.846" y="46.736" rot="MR90"/>
+<element name="R5" library="HyTechDevices" package="AXIAL-0.3EZ" value="430k" x="37.338" y="43.942" rot="MR90"/>
 <element name="U$1" library="HyTechDevices" package="SOT223" value="" x="15.24" y="10.16" rot="MR180"/>
 <element name="U$2" library="HyTechDevices" package="SOP04" value="CPC1002N" x="24.13" y="16.51" rot="MR270"/>
@@
 <wire x1="36.83" y1="55.372" x2="22.86" y2="55.372" width="0.6096" layer="16"/>
 <wire x1="36.83" y1="53.34" x2="30.85" y2="53.34" width="0.6096" layer="16"/>
-<wire x1="30.85" y1="53.34" x2="30.85" y2="47.636" width="0.6096" layer="16"/>
-<wire x1="30.85" y1="47.636" x2="30.85" y2="45.974" width="0.6096" layer="16"/>
+<wire x1="30.85" y1="53.34" x2="30.85" y2="45.974" width="0.6096" layer="16"/>
 <wire x1="22.098" y1="45.974" x2="30.85" y2="45.974" width="0.6096" layer="16"/>
 <wire x1="4.512" y1="22.479" x2="4.318" y2="22.479" width="0.6096" layer="16"/>
@@
 <wire x1="8.89" y1="55.372" x2="22.86" y2="55.372" width="0.6096" layer="16"/>
 <wire x1="9.398" y1="25.908" x2="12.446" y2="22.86" width="0.6096" layer="16"/>
-<wire x1="35.052" y1="47.636" x2="30.85" y2="47.636" width="0.6096" layer="16"/>
 <wire x1="19.05" y1="22.86" x2="16.51" y2="22.86" width="0.6096" layer="16"/>
 <wire x1="27.548" y1="35.052" x2="25.792" y2="35.052" width="0.6096" layer="16"/>
@@
 <wire x1="4.318" y1="46.99" x2="4.318" y2="22.479" width="0.6096" layer="16"/>
 <wire x1="22.098" y1="45.974" x2="22.098" y2="36.83" width="0.6096" layer="16"/>
+<wire x1="33.782" y1="45.974" x2="30.85" y2="45.974" width="0.6096" layer="16"/>
 </signal>
 <signal name="12VSUPPLY">
@@
 <contactref element="BRAKE" pad="1"/>
 <contactref element="U$4" pad="8"/>
-<contactref element="R5" pad="2"/>
+<contactref element="R5" pad="P$2"/>
 <contactref element="CALIBRATE3" pad="1"/>
 <wire x1="21.53" y1="10.795" x2="17.54" y2="10.795" width="0.6096" layer="16"/>
@@
 <wire x1="13.716" y1="27.94" x2="16.51" y2="27.94" width="0.6096" layer="16"/>
 <wire x1="16.51" y1="27.94" x2="20.622" y2="27.94" width="0.6096" layer="16"/>
-<wire x1="37.846" y1="47.636" x2="41.91" y2="47.636" width="0.6096" layer="16"/>
-<wire x1="41.91" y1="47.636" x2="41.91" y2="53.34" width="0.6096" layer="16"/>
 <wire x1="33.02" y1="30.48" x2="37.338" y2="30.48" width="0.6096" layer="16"/>
-<wire x1="37.338" y1="30.48" x2="37.338" y2="42.418" width="0.6096" layer="16"/>
-<wire x1="37.338" y1="42.418" x2="41.91" y2="42.418" width="0.6096" layer="16"/>
-<wire x1="41.91" y1="42.418" x2="41.91" y2="47.636" width="0.6096" layer="16"/>
+<wire x1="37.338" y1="30.48" x2="37.338" y2="38.1" width="0.6096" layer="16"/>
+<wire x1="37.338" y1="38.1" x2="41.91" y2="38.1" width="0.6096" layer="16"/>
+<wire x1="41.91" y1="38.1" x2="41.91" y2="47.752" width="0.6096" layer="16"/>
+<wire x1="41.91" y1="47.752" x2="41.91" y2="53.34" width="0.6096" layer="16"/>
 <wire x1="21.13" y1="17.78" x2="20.574" y2="17.78" width="0.6096" layer="16"/>
 <wire x1="20.574" y1="17.78" x2="20.574" y2="20.574" width="0.6096" layer="16"/>
@@
 <wire x1="17.272" y1="33.528" x2="13.97" y2="33.528" width="0.6096" layer="16"/>
 <wire x1="13.97" y1="33.528" x2="13.716" y2="33.274" width="0.6096" layer="16"/>
+<wire x1="37.338" y1="47.752" x2="41.91" y2="47.752" width="0.6096" layer="16"/>
 </signal>
 <signal name="N$3">
@@
 <wire x1="7.874" y1="22.479" x2="7.874" y2="45.212" width="0.6096" layer="16"/>
 <via x="7.874" y="45.212" extent="1-16" drill="0.6" shape="square"/>
-<wire x1="7.874" y1="45.212" x2="22.352" y2="45.212" width="0.6096" layer="1"/>
-<wire x1="22.352" y1="45.212" x2="25.654" y2="41.91" width="0.6096" layer="1"/>
-<via x="25.654" y="41.91" extent="1-16" drill="0.6" shape="square"/>
-<wire x1="25.654" y1="41.91" x2="35.052" y2="41.91" width="0.6096" layer="16"/>
-<wire x1="35.052" y1="41.91" x2="35.052" y2="42.026" width="0.6096" layer="16"/>
+<wire x1="7.874" y1="45.212" x2="24.13" y2="45.212" width="0.6096" layer="1"/>
+<wire x1="33.782" y1="38.978" x2="30.734" y2="38.978" width="0.6096" layer="16"/>
+<wire x1="30.734" y1="38.978" x2="30.734" y2="43.942" width="0.6096" layer="16"/>
+<wire x1="30.734" y1="43.942" x2="25.4" y2="43.942" width="0.6096" layer="16"/>
+<via x="25.4" y="43.942" extent="1-16" drill="0.6" shape="square"/>
+<wire x1="25.4" y1="43.942" x2="24.13" y2="45.212" width="0.6096" layer="1"/>
 </signal>
 <signal name="N$9">
@@
 </signal>
 <signal name="N$13">
-<contactref element="R5" pad="1"/>
+<contactref element="R5" pad="P$1"/>
 <contactref element="R3" pad="2"/>
 <contactref element="C1" pad="1"/>
 <contactref element="U$4" pad="3"/>
-<wire x1="37.846" y1="45.836" x2="35.052" y2="45.836" width="0.6096" layer="16"/>
-<wire x1="35.052" y1="45.836" x2="35.052" y2="43.826" width="0.6096" layer="16"/>
 <wire x1="26.73" y1="8.255" x2="29.464" y2="8.255" width="0.6096" layer="16"/>
 <wire x1="29.464" y1="8.255" x2="29.464" y2="8.128" width="0.6096" layer="16"/>
@@
 <wire x1="48.006" y1="8.128" x2="48.006" y2="44.196" width="0.6096" layer="16"/>
 <via x="48.006" y="44.196" extent="1-16" drill="0.6" shape="square"/>
-<wire x1="48.006" y1="44.196" x2="37.846" y2="44.196" width="0.6096" layer="1"/>
-<via x="37.846" y="44.196" extent="1-16" drill="0.6" shape="square"/>
-<wire x1="37.846" y1="44.196" x2="37.846" y2="45.836" width="0.6096" layer="16"/>
+<wire x1="48.006" y1="44.196" x2="39.878" y2="44.196" width="0.6096" layer="1"/>
+<via x="39.878" y="44.196" extent="1-16" drill="0.6" shape="square"/>
+<wire x1="37.338" y1="40.132" x2="39.878" y2="40.132" width="0.6096" layer="16"/>
+<wire x1="39.878" y1="40.132" x2="39.878" y2="43.434" width="0.6096" layer="16"/>
+<wire x1="39.878" y1="43.688" x2="39.878" y2="44.196" width="0.6096" layer="16"/>
+<wire x1="33.782" y1="40.778" x2="33.782" y2="43.434" width="0.6096" layer="16"/>
+<wire x1="33.782" y1="43.434" x2="39.878" y2="43.434" width="0.6096" layer="16"/>
+<wire x1="39.878" y1="43.434" x2="39.878" y2="43.688" width="0.6096" layer="16"/>
 </signal>
 <signal name="N$7">
@@
 <contactref element="CALIBRATE3" pad="2"/>
 <wire x1="39.37" y1="53.34" x2="39.37" y2="55.372" width="0.6096" layer="16"/>
-<wire x1="39.37" y1="55.372" x2="44.958" y2="55.372" width="0.6096" layer="16"/>
-<wire x1="44.958" y1="55.372" x2="44.958" y2="42.418" width="0.6096" layer="16"/>
+<wire x1="39.37" y1="55.372" x2="44.196" y2="55.372" width="0.6096" layer="16"/>
+<wire x1="44.196" y1="55.372" x2="44.196" y2="42.418" width="0.6096" layer="16"/>
 <via x="29.464" y="10.922" extent="1-16" drill="0.6" shape="square"/>
 <wire x1="29.464" y1="10.922" x2="46.228" y2="10.922" width="0.6096" layer="1"/>
 <via x="46.228" y="10.922" extent="1-16" drill="0.6" shape="square"/>
 <wire x1="46.228" y1="10.922" x2="46.228" y2="42.418" width="0.6096" layer="16"/>
-<wire x1="46.228" y1="42.418" x2="44.958" y2="42.418" width="0.6096" layer="16"/>
+<wire x1="46.228" y1="42.418" x2="44.196" y2="42.418" width="0.6096" layer="16"/>
 <wire x1="26.73" y1="9.525" x2="28.067" y2="9.525" width="0.6096" layer="16"/>
 <wire x1="28.067" y1="9.525" x2="29.464" y2="10.922" width="0.6096" layer="16"/>
