File: ECU-Designs/Pedal Box Board/Pedal Box Board rev1.sch (EAGLE design)
At the start: 15 parts, among them X1 MINIFIT_5566-4, X2 MINIFIT_5566-4, X3 MINIFIT_5566-10

Commit message: Modified BSPD to facilitate the reading of a rising edge trigger
Connections:
- net +5V: now also R1.1
- net N$14: no longer R3.2
- net N$3: now also R3.2
- net N$4: now also R1.2

Commit message: Add software shutdown relay to pedal box board
Parts:
- added R6: 100, HyTechDevices:RESISTOR0805-RES
- added U$4: ORWH-SH-112D1F, HyTechDevices:ORWH-SH-112D1F
- added U$5: CPC1002N, HyTechDevices:CPC1002N
Connections:
- net N$11 renamed FAULT_INDICATE
- net N$12 renamed SIGNAL_BRAKE
- net N$20 renamed READ_CHARGE
- net N$21 renamed READ_IMPED
- net N$6 renamed SIGNAL_CURRENT
- removed net N$10: X3-1.S
- new net 12VSUPPLY: U$2.IN, U$5.DC+, X1-1.S, X2-1.S, X3-9.S
- new net N$17: U$4.S, X3-1.S
- new net N$18: U$4.COIL+, U$5.DC-
- new net N$22: R6.2, U$5.CONTROL-
- new net SENSE_A: U$5.S
- new net SHUTDOWN_B: U$4.P
- new net SHUTDOWN_C: X3-2.S
- new net SHUTDOWN_RELAY_CTRL: U$1.D12, U$5.CONTROL+
- net +5V: now also R6.1, U$4.VCC
- net GND: now also R6.1, U$4.COIL-, U$4.GND
- net N$1: no longer U$2.IN, X1-1.S, X2-1.S, X3-9.S
- net N$13: now also U$4.1IN+; no longer X3-2.S
- net N$7: now also U$4.1IN-
- net N$9: now also R6.2, U$4.1OUT
Other:
- moved on the sheet: X3-1, X3-10, X3-2, X3-3, X3-4, X3-5, X3-6, X3-7, X3-8, X3-9

Commit message: Add voltage dividers to pedal sensor outputs
Parts:
- added R10, R11, R12: 15k, HyTechDevices:RESISTOR0805-RES
- added R7, R8, R9: 10k, HyTechDevices:RESISTOR0805-RES
- R5: device HyTechDevices:RESISTOREZ -> HyTechDevices:RESISTORPTH-1/4W-VERT
Connections:
- new net N$10: R12.2, R9.2, U$1.A2
- new net N$6: R11.2, R8.2, U$1.A1
- net GND: now also R10.1, R11.1, R12.1
- net N$1: now also PEDALS-9.S, R7.1
- net N$7: now also R5.2, R9.1; no longer R5.1, U$1.A2
- net N$8: now also R8.1; no longer U$1.A1
- net N$9: now also R10.2, R7.2; no longer PEDALS-9.S
- net SIGNAL_BRAKE: now also R5.1; no longer R5.2
Other:
- note added: "Voltage dividers"
- moved on the sheet: PEDALS-1, PEDALS-10, PEDALS-2, PEDALS-3, PEDALS-4, PEDALS-5, PEDALS-6, PEDALS-7, PEDALS-8, PEDALS-9, R5, U$3

Commit message: Update smart precharger symbol, add crash sensor symbol, update shutdown circuit
Parts:
- added D1: DIODE0805, HyTechDevices:DIODE0805
Connections:
- net N$17 renamed SHUTDOWN_A
- removed net SENSE_A: U$5.S
- removed net SENSE_B: U$1.S
- removed net SHUTDOWN_IN: U$3.6
- removed net SHUTDOWN_OUT: U$3.7
- new net N$11: D1.A, PEDALS-3.S, R5.2
- net N$7: now also D1.C; no longer PEDALS-3.S, R5.2
- net SHUTDOWN_B: now also U$3.6
- net SHUTDOWN_C: now also U$3.7
Other:
- note added: "TODO check FSAE EV5.1.6"
- moved on the sheet: PEDALS-1, PEDALS-10, PEDALS-2, PEDALS-3, PEDALS-4, PEDALS-5, PEDALS-6, PEDALS-7, PEDALS-8, PEDALS-9

Commit message: Add FSAE EV5.1.6 compliance to BSPD
Connections:
- new net SHUTDOWN_D: U$3.7
- net +5V: now also U$1.COIL-
- net GND: now also U$1.COIL+
- net N$2: now also U$1.S, U$3.6
- net SHUTDOWN_B: now also U$1.P; no longer U$3.6
- net SHUTDOWN_C: no longer U$3.7
Other:
- note added: "Normally Open Relay -> FSAE EV5.1.6"

Commit message: Make bspd layout more efficient, change relays used, add Omron G5LE Relay to library
Parts:
- U$4: value ORWH-SH-112D1F -> G5LE; device HyTechDevices:ORWH-SH-112D1F -> HyTechDevices:G5LE
Connections:
- net FAULT_INDICATE renamed READ_FAULT
- net READ_IMPED renamed READ_SWITCH
- removed net 12VSUPPLY: U$2.IN, U$5.DC+, X1-1.S, X2-1.S, X3-9.S
- new net +12V: U$1.COIL-, U$2.IN, U$5.DC+, X1-1.S, X2-1.S, X3-9.S
- net +5V: no longer U$1.COIL-
- net N$10: now also R1.2
- net N$3: no longer R3.2
- net N$4: now also R3.2; no longer R1.2
Other:
- note removed: "TODO check FSAE EV5.1.6"

Commit message: Finish BSPD/throttle board layout
Parts:
- removed U$4: G5LE, HyTechDevices:G5LE
- added SOFTWARE_SHUTOFF: G5LE, HyTechDevices:G5LE
- renumbered X3 to BSPD
Connections:
- removed net N$18: U$4.COIL+, U$5.DC-
- new net N$12: SOFTWARE_SHUTOFF.COIL-, U$5.DC-
- net +5V: no longer U$4.VCC
- net GND: now also SOFTWARE_SHUTOFF.COIL+; no longer U$4.COIL-, U$4.GND
- net N$13: no longer U$4.1IN+
- net N$2: no longer U$1.S, U$3.6
- net N$7: no longer U$4.1IN-
- net N$9: no longer U$4.1OUT
- net SHUTDOWN_A: now also SOFTWARE_SHUTOFF.P; no longer U$4.S
- net SHUTDOWN_B: now also SOFTWARE_SHUTOFF.S; no longer U$4.P
- net SHUTDOWN_C: now also U$1.S, U$3.6; no longer BSPD-2.S
- net SHUTDOWN_D: now also BSPD-2.S

Commit message: Pedal box board
Parts:
- R2, R3, R4: value (none) -> 150
Changed lines of the file:
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@@
 <part name="LED2" library="HyTechDevices" deviceset="LED" device="-0805"/>
 <part name="LED3" library="HyTechDevices" deviceset="LED" device="-0805"/>
-<part name="R2" library="HyTechDevices" deviceset="RESISTOR" device="0805-RES"/>
-<part name="R3" library="HyTechDevices" deviceset="RESISTOR" device="0805-RES"/>
-<part name="R4" library="HyTechDevices" deviceset="RESISTOR" device="0805-RES"/>
+<part name="R2" library="HyTechDevices" deviceset="RESISTOR" device="0805-RES" value="150"/>
+<part name="R3" library="HyTechDevices" deviceset="RESISTOR" device="0805-RES" value="150"/>
+<part name="R4" library="HyTechDevices" deviceset="RESISTOR" device="0805-RES" value="150"/>
 <part name="GND8" library="HyTechSymbols" deviceset="GND" device=""/>
 <part name="R5" library="HyTechDevices" deviceset="RESISTOR" device="PTH-1/4W-VERT" value="JMP"/>
