File: ECU-Designs/Pedal Box Board/Pedal Box Board rev3.brd (EAGLE design)
At the start: 107.2 x 139.4 mm, 66 parts, among them X1 MINIFIT_5566-4, X2 MINIFIT_5566-4, X3 CONNECTOR-4MX150L_VERTICAL-4, X4 CONNECTOR-10MX150L_VERTICAL-10, X5 CONNECTOR-10MX150L_VERTICAL-10, X6 CONNECTOR-10MX150L_VERTICAL-10

Commit message: Add some new boards and revisions, schematics for ESF, deleted HyTechDevices2
Parts:
- turned X3 to 270 degrees
Routing:
- net GND: track 651.8 -> 681.2 mm
- net N$4: track 109.8 -> 91.6 mm
- net +12V: track 414.4 -> 428.6 mm
- net SHUTDOWN_A: track 227.4 -> 233.1 mm
- net N$3: track 75.0 -> 71.5 mm
Changed lines of the file:
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@@
 <element name="BSPD1:D1" library="HyTechDevices" package="0805_D" value="DIODE0805" x="81.788" y="89.916" rot="MR270"/>
 <element name="BSPD1:D2" library="HyTechDevices" package="0805_D" value="DIODE0805" x="85.852" y="44.196" rot="MR270"/>
-<element name="X3" library="HyTechDevices" package="MX150L_VERTICAL-4" value="CONNECTOR-4MX150L_VERTICAL-4" x="17.272" y="106.172" rot="MR90"/>
+<element name="X3" library="HyTechDevices" package="MX150L_VERTICAL-4" value="CONNECTOR-4MX150L_VERTICAL-4" x="17.272" y="106.172" rot="MR270"/>
 <element name="X4" library="HyTechDevices" package="MX150L_VERTICAL-10" value="CONNECTOR-10MX150L_VERTICAL-10" x="69.596" y="18.796" rot="MR0"/>
 <element name="X5" library="HyTechDevices" package="MX150L_VERTICAL-10" value="CONNECTOR-10MX150L_VERTICAL-10" x="69.088" y="122.936" rot="MR180"/>
@@
 <wire x1="37.846" y1="92.71" x2="37.846" y2="87.19" width="0.4064" layer="16"/>
 <contactref element="X3" pad="3"/>
-<wire x1="14.2748" y1="103.251" x2="17.6149" y2="99.9109" width="0.6096" layer="1"/>
-<wire x1="30.6451" y1="99.9109" x2="37.846" y2="92.71" width="0.6096" layer="1"/>
 <via x="37.846" y="92.71" extent="1-16" drill="0.6" shape="square"/>
-<wire x1="17.6149" y1="99.9109" x2="30.6451" y2="99.9109" width="0.6096" layer="1"/>
-<wire x1="37.846" y1="92.71" x2="44.704" y2="92.71" width="0.4064" layer="1"/>
+<wire x1="44.704" y1="92.71" x2="37.846" y2="92.71" width="0.4064" layer="1"/>
 <wire x1="44.704" y1="92.71" x2="45.974" y2="91.44" width="0.4064" layer="1"/>
 <contactref element="X2" pad="3"/>
@@
 <wire x1="35.814" y1="74.49" x2="37.89" y2="74.49" width="0.4064" layer="16"/>
 <wire x1="35.814" y1="87.19" x2="35.814" y2="74.49" width="0.4064" layer="16"/>
+<wire x1="21.463" y1="109.093" x2="20.2692" y2="109.093" width="0.6096" layer="1"/>
+<wire x1="37.846" y1="92.71" x2="21.463" y2="109.093" width="0.6096" layer="1"/>
 <wire x1="37.89" y1="87.19" x2="37.846" y2="87.19" width="0" layer="19" extent="16-16"/>
 </signal>
@@
 <wire x1="37.89" y1="70.29" x2="34.544" y2="70.29" width="0.4064" layer="16"/>
 <contactref element="X3" pad="4"/>
-<wire x1="10.16" y1="104.9782" x2="14.2748" y2="109.093" width="0.6096" layer="1"/>
 <wire x1="37.89" y1="82.99" x2="37.89" y2="85.09" width="0.4064" layer="16"/>
 <wire x1="37.89" y1="85.09" x2="37.846" y2="85.09" width="0.4064" layer="16"/>
@@
 <wire x1="45.466" y1="80.772" x2="37.846" y2="80.772" width="0.4064" layer="1"/>
 <wire x1="37.846" y1="80.772" x2="32.258" y2="80.772" width="0.6096" layer="1"/>
-<wire x1="10.16" y1="101.6" x2="10.16" y2="104.9782" width="0.6096" layer="1"/>
-<wire x1="27.559" y1="95.123" x2="24.511" y2="98.171" width="0.6096" layer="1"/>
-<wire x1="24.511" y1="98.171" x2="13.589" y2="98.171" width="0.6096" layer="1"/>
-<wire x1="13.589" y1="98.171" x2="10.16" y2="101.6" width="0.6096" layer="1"/>
 <wire x1="27.559" y1="85.471" x2="27.559" y2="95.123" width="0.6096" layer="1"/>
 <wire x1="32.258" y1="80.772" x2="27.559" y2="85.471" width="0.6096" layer="1"/>
+<wire x1="20.2692" y1="102.4128" x2="20.2692" y2="103.251" width="0.6096" layer="1"/>
+<wire x1="27.559" y1="95.123" x2="20.2692" y2="102.4128" width="0.6096" layer="1"/>
 </signal>
 <signal name="GND">
@@
 <wire x1="37.846" y1="67.818" x2="40.64" y2="67.818" width="0.6096" layer="16"/>
 <wire x1="41.275" y1="96.774" x2="40.894" y2="96.774" width="0.6096" layer="16"/>
-<wire x1="20.2692" y1="109.093" x2="40.894" y2="109.093" width="1.778" layer="1"/>
 <wire x1="49.276" y1="102.87" x2="49.276" y2="108.966" width="0.6096" layer="16"/>
 <via x="40.894" y="96.774" extent="1-16" drill="0.6" shape="square"/>
-<wire x1="40.894" y1="109.093" x2="40.894" y2="96.774" width="1.778" layer="1"/>
+<wire x1="40.894" y1="96.774" x2="40.894" y2="109.093" width="1.778" layer="1"/>
 <via x="40.894" y="109.093" extent="1-16" drill="0.6" shape="square"/>
 <wire x1="49.276" y1="108.966" x2="40.894" y2="108.966" width="0.6096" layer="16"/>
@@
 <wire x1="27.94" y1="60.452" x2="28.702" y2="59.69" width="0.4064" layer="1"/>
 <wire x1="28.702" y1="59.69" x2="28.702" y2="58.801" width="0.4064" layer="1"/>
+<wire x1="40.894" y1="109.093" x2="31.623" y2="109.093" width="1.778" layer="1"/>
+<wire x1="25.4" y1="115.316" x2="9.906" y2="115.316" width="1.778" layer="1"/>
+<wire x1="9.906" y1="115.316" x2="9.906" y2="103.251" width="1.778" layer="1"/>
+<wire x1="9.906" y1="103.251" x2="14.2748" y2="103.251" width="1.778" layer="1"/>
+<wire x1="31.623" y1="109.093" x2="25.4" y2="115.316" width="1.778" layer="1"/>
 </signal>
 <signal name="+5V">
@@
 <wire x1="57.404" y1="111.252" x2="46.482" y2="111.252" width="1.778" layer="1"/>
 <wire x1="51.816" y1="58.42" x2="37.592" y2="58.42" width="1.778" layer="1"/>
-<wire x1="6.35" y1="101.092" x2="6.35" y2="113.792" width="1.778" layer="1"/>
 <wire x1="46.482" y1="111.252" x2="43.942" y2="113.792" width="1.778" layer="1"/>
-<wire x1="43.942" y1="113.792" x2="6.35" y2="113.792" width="1.778" layer="1"/>
+<wire x1="43.942" y1="113.792" x2="33.782" y2="113.792" width="1.778" layer="1"/>
 <wire x1="25.146" y1="92.71" x2="25.146" y2="77.216" width="1.778" layer="1"/>
 <wire x1="25.146" y1="92.71" x2="22.606" y2="95.25" width="1.778" layer="1"/>
 <wire x1="22.606" y1="95.25" x2="12.192" y2="95.25" width="1.778" layer="1"/>
-<wire x1="12.192" y1="95.25" x2="6.35" y2="101.092" width="1.778" layer="1"/>
+<wire x1="6.35" y1="101.092" x2="12.192" y2="95.25" width="1.778" layer="1"/>
 <wire x1="33.02" y1="62.992" x2="33.02" y2="69.342" width="1.778" layer="1"/>
 <wire x1="25.146" y1="77.216" x2="33.02" y2="69.342" width="1.778" layer="1"/>
@@
 <wire x1="57.912" y1="65.278" x2="58.928" y2="64.262" width="0.4064" layer="16"/>
 <wire x1="58.928" y1="64.262" x2="58.928" y2="58.42" width="0.4064" layer="16"/>
+<wire x1="29.718" y1="117.856" x2="6.35" y2="117.856" width="1.778" layer="1"/>
+<wire x1="33.782" y1="113.792" x2="29.718" y2="117.856" width="1.778" layer="1"/>
+<wire x1="6.35" y1="117.856" x2="6.35" y2="101.092" width="1.778" layer="1"/>
 </signal>
 <signal name="SHUTDOWN_RELAY_CTRL">
@@
 <wire x1="31.242" y1="72.644" x2="31.242" y2="78.486" width="0.4064" layer="16"/>
 <wire x1="46.228" y1="74.49" x2="46.228" y2="78.74" width="1.778" layer="16"/>
-<wire x1="20.2692" y1="103.251" x2="20.3962" y2="103.124" width="1.778" layer="1"/>
-<wire x1="20.3962" y1="103.124" x2="31.242" y2="103.124" width="1.778" layer="1"/>
 <wire x1="27.686" y1="54.991" x2="25.273" y2="54.991" width="0.4064" layer="1"/>
 <wire x1="25.273" y1="57.531" x2="27.686" y2="57.531" width="0.4064" layer="1"/>
@@
 <wire x1="27.686" y1="58.928" x2="26.924" y2="59.69" width="0.4064" layer="1"/>
 <wire x1="27.686" y1="57.531" x2="27.686" y2="58.928" width="0.4064" layer="1"/>
+<wire x1="14.2748" y1="109.093" x2="14.2748" y2="112.776" width="1.778" layer="1"/>
+<wire x1="31.242" y1="104.14" x2="31.242" y2="103.124" width="1.778" layer="1"/>
+<wire x1="14.2748" y1="112.776" x2="22.606" y2="112.776" width="1.778" layer="1"/>
+<wire x1="22.606" y1="112.776" x2="31.242" y2="104.14" width="1.778" layer="1"/>
 </signal>
 <signal name="BSPD1:N$10">
