File: ECU-Designs/BMS-ECU/BMS Segment Jeff v1.sch (EAGLE design)
At the start: 68 parts, among them T1 NPN_BCP56T1, X1 MINIFIT_5566-2, X2 To Positive BMS

Commit message: Finished Negative Side BMS Board Layout
Parts:
- removed ISOSPI_IN, ISOSPI_OUT, X1: MINIFIT_5566-2, HyTechDevices:MINIFIT_5566-2
- removed SENSE_LINES: MINIFIT_5566-4, HyTechDevices:MINIFIT_5566-4
- removed X2: To Positive BMS, HyTechDevices:MINIFIT_5566-2
- added BMSIN, BMSOUT: CONNECTOR-4NANO-FIT-VERTICAL-4, HyTechDevices:CONNECTOR-4NANO-FIT-VERTICAL-4
- added TO_TOP: CONNECTOR-2NANO-FIT_VERTICAL-2, HyTechDevices:CONNECTOR-2NANO-FIT_VERTICAL-2
- added X3: Th1, HyTechDevices:CONNECTOR-2NANO-FIT_VERTICAL-2
- added X4: Th2, HyTechDevices:CONNECTOR-2NANO-FIT_VERTICAL-2
- added X5: Th3, HyTechDevices:CONNECTOR-2NANO-FIT_VERTICAL-2
Connections:
- removed net CURRENT_SENSE: SENSE_LINES-4.S, U$2.GPI04
- removed net SSR+: GLV_CONTROL.CONTROL+, X1-1.S
- new net SHUTDOWN_CIRCUIT: BMSIN-1.S, BMSOUT-1.S, GLV_CONTROL.CONTROL+
- net GND: now also BMSIN-2.S, BMSOUT-2.S; no longer X1-2.S
- net ISOSPI-M_IN: now also BMSIN-3.S; no longer ISOSPI_IN-2.S
- net ISOSPI-M_OUT: now also BMSOUT-3.S; no longer ISOSPI_OUT-2.S
- net ISOSPI-P_IN: now also BMSIN-4.S; no longer ISOSPI_IN-1.S
- net ISOSPI-P_OUT: now also BMSOUT-4.S; no longer ISOSPI_OUT-1.S
- net SENSE9: now also TO_TOP-1.S, TO_TOP-2.S; no longer X2-1.S, X2-2.S
- net THERMISTOR1: now also R101.2, X5-2.S; no longer R103.2, SENSE_LINES-1.S
- net THERMISTOR2: now also X4-2.S; no longer SENSE_LINES-2.S
- net THERMISTOR3: now also R103.2, X3-2.S; no longer R101.2, SENSE_LINES-3.S
- net V-: now also X3-1.S, X4-1.S, X5-1.S
Other:
- note added: "Total of 6 termistors per 18 cell segment"
- note removed: "From previous module"
- note removed: "To next module"
- moved on the sheet: R102, R103
