File: ECU-Designs/HV Box/HV-main rev0 Manufactured 2017-04-01.brd (EAGLE design)
At the start: 196.1 x 63.5 mm, 68 parts, among them IC2 MCP6002SOIC, IC3 MCP6002SOIC

Commit message: Move files, upload final designs with logos, update jeff bms layout for rules compliance
Other:
- board text added: "hv_board_rev0"
- board text removed: "hv_board_rev1"
Changed lines of the file:
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@@
 <text x="186.436" y="7.112" size="2.1844" layer="52" rot="MR270">GLV</text>
 <text x="188.976" y="7.112" size="2.1844" layer="52" rot="MR90" align="bottom-right">TS</text>
-<text x="220.98" y="27.94" size="1.27" layer="52" font="vector" rot="R270">hv_board_rev1</text>
+<text x="220.98" y="27.94" size="1.27" layer="52" font="vector" rot="R270">hv_board_rev0</text>
 <rectangle x1="67.1322" y1="13.0302" x2="68.5038" y2="13.1064" layer="51" rot="R90"/>
 <rectangle x1="67.0179" y1="16.1925" x2="68.6181" y2="16.2687" layer="51" rot="R90"/>
