File: Tractive System Diagram.sch (EAGLE design)
At the start: 15 parts

Commit message: Update ts schematic, separate shutdown circuits for FH and FSAE, add Aaron's changes to BMS test board
Parts:
- removed MOLEX_IMPERIUM_INTERLOCK: SWITCH_SPST, HyTechSymbols:SWITCH_SPST
- added EMRAX_207_MED_V_MOTOR: MOTOR_AC, HyTechSymbols:MOTOR_AC
- added FUSE: 200A, HyTechSymbols:FUSE
- added INTERLOCK: SWITCH_SPST, HyTechSymbols:SWITCH_SPST
- added MOLEX_IMPERIUM1: (no value), HyTechSymbols:M02
- added SEGMENT1, SEGMENT2, SEGMENT3, SEGMENT4: BATTERY_1_CELL, HyTechSymbols:BATTERY_1_CELL
- added U$2: RINEHART_PM100DX, HyTechSymbols:RINEHART_PM100DX
Connections:
- removed net N$10: AIR2.S
- removed net N$12: AIR2.P, HV_FUSE2.1, MOLEX_IMPERIUM.2
- removed net N$19: MOLEX_IMPERIUM_INTERLOCK.S, SL1.1
- removed net N$3: AIR1.P, U$1.CTCS+
- removed net N$4: SMD1.S
- removed net N$5: SMD1.P
- removed net N$6: SMD2.S
- removed net N$7: SMD2.P
- removed net N$8: SMD3.S
- removed net N$9: SMD3.P
- new net N$1: HV_FUSE1.1
- new net N$2: HV_FUSE2.1
- new net SHUTDOWN_CIRCUIT_POST_INTERLOCK: AIR2.2, INTERLOCK.P, SMD1.2, SMD2.2, SMD3.2, U$1.12V
- new net SHUTDOWN_CIRCUIT_PRE_INTERLOCK: INTERLOCK.S, SL1.1
- net GND: now also AIR2.1; no longer AIR2.2
- net N$11: no longer AIR1.S, HV_FUSE1.1, MOLEX_IMPERIUM.1
- net N$13: now also U$1.CTCS+; no longer AIR2.1, MOLEX_IMPERIUM_INTERLOCK.P, SMD1.2, SMD2.2, SMD3.2, U$1.12V
Other:
- note added: "Key Thick: High Voltage wires Orange: High Current path Blue: VSense, TSense connections"
- note added: "Molex Imperium also used for charging"
- moved on the sheet: AIR2, HV_FUSE1, HV_FUSE2, SL1, SMD1, SMD2, SMD3, TSMP+, TSMP-

Commit message: Updated TS schematic, external diagram with latest design and requirements
Parts:
- removed HV_FUSE1, HV_FUSE2: (no value), HyTechSymbols:FUSE
- added PCB_F1, PCB_F2, PC_F1, PC_F2: 6.3A, HyTechSymbols:FUSE
- added TSMP+1, TSMP+2, TSMP-1, TSMP-2: 5k, HyTechDevices:RESISTOR10W
Connections:
- new net HV+: PCB_F1.1, TSMP+1.2
- new net HV-: PCB_F2.1, TSMP-1.2
- new net N$10: U$4.XLA-(HV-)
- new net N$12: U$4.XLA+(HV+)
- new net N$35: PC_F1.2, U$1.CTCS+
- new net N$36: PC_F2.2, U$1.CTCS-
- net GND: now also AIR1.1; no longer AIR2.1
- net N$1: now also TSMP+1.1, TSMP+2.2; no longer HV_FUSE1.1
- net N$11: now also PC_F2.1; no longer U$1.CTCS-
- net N$13: now also PC_F1.1; no longer U$1.CTCS+
- net N$14: now also TSMP+2.1
- net N$16: now also TSMP-2.1
- net N$2: now also TSMP-1.1, TSMP-2.2; no longer HV_FUSE2.1
- net N$20: now also AIR2.2; no longer AIR1.2
- net N$21: now also AIR2.1; no longer AIR1.1
- net N$22: now also PCB_F1.2; no longer HV_FUSE1.2, U$4.XLA+(HV+)
- net N$24: now also PCB_F2.2; no longer HV_FUSE2.2, U$4.XLA-(HV-)
- net SHUTDOWN_CIRCUIT_POST_INTERLOCK: now also AIR1.2; no longer AIR2.2
Other:
- note added: "2 10W 5kΩ resistors in series"
- note added: "TODO Add Energy Meter"
- note added: "TODO fix ports on HV_PCB"
- note added: "Wire Key Thick: High Voltage wires Orange: High Current path Blue: VSense, TSense connections"
- note removed: "Key Thick: High Voltage wires Orange: High Current path Blue: VSense, TSense connections"
- moved on the sheet: ACCUMULATOR_INDICATOR, AIR1, AIR2, FUSE, SEGMENT1, SEGMENT2, SEGMENT3, SEGMENT4, SL1, SMD1, SMD2, SMD3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

Commit message: Add discharge resistor, fix I/O on tractive system schematic
Parts:
- added DISCHARGE: (no value), HyTechDevices:RESISTOR10W
- added SL2: (no value), HyTechSymbols:M04
- SL1: device HyTechSymbols:M11 -> HyTechSymbols:M09
Connections:
- removed net N$25 (its old number): SL1.10
- new net N$27: SL1.4
- new net N$30: SL1.7
- new net N$38: DISCHARGE.2
- new net N$39: DISCHARGE.1
- new net N$43: SL2.1
- new net N$44: SL2.2
- new net N$45: SL2.3
- new net N$46: SL2.4
- net N$23: now also SL1.1; no longer SL1.11
- net SHUTDOWN_CIRCUIT_PRE_INTERLOCK: no longer SL1.1
Other:
- note added: "Wire Key Thick: Tractive System wires Orange: High Current path Blue: VSense, TSense connections"
- note removed: "TODO fix ports on HV_PCB"
- note removed: "Wire Key Thick: High Voltage wires Orange: High Current path Blue: VSense, TSense connections"
- moved on the sheet: ACCUMULATOR_INDICATOR, PCB_F1, PCB_F2, TSMP+2, TSMP-2

Commit message: Add energy meter to tractive system diagram
Parts:
- added SL3: (no value), HyTechSymbols:M02
Connections:
- new net N$51: SL3.1
- new net N$52: SL3.2
Other:
- note added: "FSAE Energy Meter (internal busbar bypass for FH)"
- note added: "HVD"
- note removed: "TODO Add Energy Meter"
- moved on the sheet: EMRAX_207_MED_V_MOTOR
Changed lines of the file:
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@@
+</sheets>
+</module>
+<module name="FSAE_ENERGY_METER" prefix="" dx="35.56" dy="20.32">
+<ports>
+<port name="HV-OUT" side="left" coord="5.08" direction="nc"/>
+<port name="HV+OUT" side="left" coord="-5.08" direction="nc"/>
+<port name="HV-IN" side="right" coord="5.08" direction="nc"/>
+<port name="HV+IN" side="right" coord="-5.08" direction="nc"/>
+<port name="12V+" side="bottom" coord="0" direction="in"/>
+<port name="GND" side="bottom" coord="2.54" direction="out"/>
+</ports>
+<variantdefs>
+</variantdefs>
+<parts>
+</parts>
+<sheets>
+<sheet>
+<plain>
+</plain>
+<instances>
+</instances>
+<busses>
+</busses>
+<nets>
+</nets>
+</sheet>
 </sheets>
 </module>
@@
 <part name="DISCHARGE" library="HyTechDevices" deviceset="RESISTOR" device="10W"/>
 <part name="SL2" library="HyTechSymbols" deviceset="M04" device=""/>
+<part name="SL3" library="HyTechSymbols" deviceset="M02" device=""/>
 </parts>
 <sheets>
@@
 <wire x1="332.74" y1="58.42" x2="332.74" y2="55.88" width="0.381" layer="156"/>
 <wire x1="335.28" y1="55.88" x2="332.74" y2="55.88" width="0.381" layer="156"/>
-<text x="223.52" y="116.84" size="2.1844" layer="91">Molex Imperium also used for charging</text>
+<text x="223.52" y="116.84" size="2.1844" layer="97">Molex Imperium also used for charging</text>
 <wire x1="345.44" y1="58.42" x2="350.52" y2="58.42" width="0.381" layer="156"/>
 <wire x1="350.52" y1="58.42" x2="350.52" y2="86.36" width="0.381" layer="156"/>
 <wire x1="350.52" y1="86.36" x2="215.9" y2="86.36" width="0.381" layer="156"/>
-<text x="304.8" y="93.98" size="2.1844" layer="91">Wire Key
+<text x="304.8" y="93.98" size="2.1844" layer="97">Wire Key
 Thick: Tractive System wires
 Orange: High Current path
 Blue: VSense, TSense connections</text>
-<wire x1="213.36" y1="121.92" x2="198.12" y2="121.92" width="0.381" layer="156"/>
-<wire x1="198.12" y1="132.08" x2="215.9" y2="132.08" width="0.381" layer="156"/>
 <wire x1="215.9" y1="132.08" x2="215.9" y2="121.92" width="0.381" layer="156"/>
-<wire x1="121.92" y1="119.38" x2="121.92" y2="114.3" width="0.381" layer="156"/>
-<wire x1="121.92" y1="114.3" x2="114.3" y2="114.3" width="0.381" layer="156"/>
-<wire x1="121.92" y1="127" x2="114.3" y2="127" width="0.381" layer="156"/>
-<wire x1="114.3" y1="139.7" x2="121.92" y2="139.7" width="0.381" layer="156"/>
-<wire x1="121.92" y1="139.7" x2="121.92" y2="134.62" width="0.381" layer="156"/>
-<text x="137.16" y="99.06" size="1.778" layer="91">2 10W 5kΩ resistors in series</text>
+<wire x1="71.12" y1="119.38" x2="71.12" y2="114.3" width="0.381" layer="156"/>
+<wire x1="71.12" y1="114.3" x2="63.5" y2="114.3" width="0.381" layer="156"/>
+<wire x1="71.12" y1="127" x2="63.5" y2="127" width="0.381" layer="156"/>
+<wire x1="63.5" y1="139.7" x2="71.12" y2="139.7" width="0.381" layer="156"/>
+<wire x1="71.12" y1="139.7" x2="71.12" y2="134.62" width="0.381" layer="156"/>
+<text x="137.16" y="96.52" size="1.778" layer="97">2 10W 5kΩ resistors in series</text>
 <wire x1="269.24" y1="58.42" x2="264.16" y2="58.42" width="0.381" layer="156"/>
-<text x="226.06" y="134.62" size="2.54" layer="91">TODO Add Energy Meter</text>
+<wire x1="147.32" y1="132.08" x2="154.94" y2="132.08" width="0.381" layer="156"/>
+<wire x1="154.94" y1="121.92" x2="147.32" y2="121.92" width="0.381" layer="156"/>
+<wire x1="200.66" y1="132.08" x2="215.9" y2="132.08" width="0.381" layer="156"/>
+<wire x1="200.66" y1="121.92" x2="213.36" y2="121.92" width="0.381" layer="156"/>
+<text x="162.56" y="139.7" size="1.778" layer="97">FSAE Energy Meter (internal busbar bypass for FH)</text>
+<text x="203.2" y="99.06" size="2.54" layer="97" rot="R90">HVD</text>
 </plain>
 <moduleinsts>
@@
 <attribute name="NAME" x="121.92" y="39.37" size="2.032" layer="95" align="bottom-center"/>
 </moduleinst>
+<moduleinst name="ENERGY_METER_BOX" module="FSAE_ENERGY_METER" x="177.8" y="127"/>
 </moduleinsts>
 <instances>
@@
 <instance part="GND5" gate="1" x="332.74" y="48.26" rot="R270"/>
 <instance part="MOLEX_IMPERIUM1" gate="G$1" x="215.9" y="116.84" rot="MR90"/>
-<instance part="U$2" gate="G$1" x="193.04" y="109.22" rot="MR0"/>
-<instance part="EMRAX_207_MED_V_MOTOR" gate="G$1" x="86.36" y="127" rot="R90"/>
+<instance part="U$2" gate="G$1" x="142.24" y="109.22" rot="MR0"/>
+<instance part="EMRAX_207_MED_V_MOTOR" gate="G$1" x="35.56" y="127" rot="R90"/>
 <instance part="TSMP+1" gate="G$1" x="124.46" y="104.14"/>
 <instance part="TSMP+2" gate="G$1" x="111.76" y="104.14"/>
@@
 <instance part="DISCHARGE" gate="G$1" x="40.64" y="91.44"/>
 <instance part="SL2" gate="G$1" x="5.08" y="48.26" rot="MR180"/>
+<instance part="SL3" gate="G$1" x="177.8" y="104.14" rot="R90"/>
 </instances>
 <busses>
@@
 </segment>
 </net>
+<net name="N$51" class="0">
+<segment>
+<portref moduleinst="ENERGY_METER_BOX" port="GND"/>
+<pinref part="SL3" gate="G$1" pin="1"/>
+<wire x1="180.34" y1="109.22" x2="180.34" y2="111.76" width="0.1524" layer="91"/>
+</segment>
+</net>
+<net name="N$52" class="0">
+<segment>
+<portref moduleinst="ENERGY_METER_BOX" port="12V+"/>
+<pinref part="SL3" gate="G$1" pin="2"/>
+<wire x1="177.8" y1="109.22" x2="177.8" y2="111.76" width="0.1524" layer="91"/>
+</segment>
+</net>

Commit message: Updates to schematics for ESFs, apparently some update to jeff bms v2
Parts:
- added HVD_INTERLOCK: SWITCH_SPST, HyTechSymbols:SWITCH_SPST
Connections:
- new net N$53: HVD_INTERLOCK.P, INTERLOCK.S
- net SHUTDOWN_CIRCUIT_PRE_INTERLOCK: now also HVD_INTERLOCK.S; no longer INTERLOCK.S

Commit message: Various updates, fix devices library
Parts:
- removed SL3: (no value), HyTechSymbols:M02
- added HVD: (no value), HyTechSymbols:M02
Connections:
- removed net N$51: SL3.1
- removed net N$52: SL3.2
Other:
- note removed: "FSAE Energy Meter (internal busbar bypass for FH)"
- note removed: "HVD"
- moved on the sheet: AIR1
Changed lines of the file:
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@@
 <part name="DISCHARGE" library="HyTechDevices" deviceset="RESISTOR" device="10W"/>
 <part name="SL2" library="HyTechSymbols" deviceset="M04" device=""/>
-<part name="SL3" library="HyTechSymbols" deviceset="M02" device=""/>
 <part name="HVD_INTERLOCK" library="HyTechSymbols" deviceset="SWITCH_SPST" device=""/>
+<part name="HVD" library="HyTechSymbols" deviceset="M02" device=""/>
 </parts>
 <sheets>
@@
 <wire x1="297.18" y1="55.88" x2="299.72" y2="55.88" width="0.381" layer="156"/>
 <wire x1="309.88" y1="58.42" x2="317.5" y2="58.42" width="0.381" layer="156"/>
-<wire x1="327.66" y1="58.42" x2="332.74" y2="58.42" width="0.381" layer="156"/>
-<wire x1="332.74" y1="58.42" x2="332.74" y2="55.88" width="0.381" layer="156"/>
-<wire x1="335.28" y1="55.88" x2="332.74" y2="55.88" width="0.381" layer="156"/>
+<wire x1="332.74" y1="58.42" x2="340.36" y2="58.42" width="0.381" layer="156"/>
+<wire x1="340.36" y1="58.42" x2="340.36" y2="55.88" width="0.381" layer="156"/>
+<wire x1="342.9" y1="55.88" x2="340.36" y2="55.88" width="0.381" layer="156"/>
 <text x="205.74" y="137.16" size="2.1844" layer="97">Molex Imperium also used for charging</text>
-<wire x1="345.44" y1="58.42" x2="350.52" y2="58.42" width="0.381" layer="156"/>
-<wire x1="350.52" y1="58.42" x2="350.52" y2="86.36" width="0.381" layer="156"/>
-<wire x1="350.52" y1="86.36" x2="215.9" y2="86.36" width="0.381" layer="156"/>
+<wire x1="353.06" y1="58.42" x2="353.06" y2="86.36" width="0.381" layer="156"/>
+<wire x1="353.06" y1="86.36" x2="215.9" y2="86.36" width="0.381" layer="156"/>
 <text x="304.8" y="93.98" size="2.1844" layer="97">Wire Key
 Thick: Tractive System wires
@@
 <text x="137.16" y="96.52" size="1.778" layer="97">2 10W 5kΩ resistors in series</text>
 <wire x1="269.24" y1="58.42" x2="264.16" y2="58.42" width="0.381" layer="156"/>
-<wire x1="147.32" y1="132.08" x2="154.94" y2="132.08" width="0.381" layer="156"/>
-<wire x1="154.94" y1="121.92" x2="147.32" y2="121.92" width="0.381" layer="156"/>
-<wire x1="200.66" y1="132.08" x2="215.9" y2="132.08" width="0.381" layer="156"/>
-<wire x1="200.66" y1="121.92" x2="213.36" y2="121.92" width="0.381" layer="156"/>
-<text x="162.56" y="139.7" size="1.778" layer="97">FSAE Energy Meter (internal busbar bypass for FH)</text>
-<text x="203.2" y="99.06" size="2.54" layer="97" rot="R90">HVD</text>
+<wire x1="147.32" y1="132.08" x2="215.9" y2="132.08" width="0.381" layer="156"/>
+<wire x1="213.36" y1="121.92" x2="147.32" y2="121.92" width="0.381" layer="156"/>
+<wire x1="330.2" y1="58.42" x2="327.66" y2="58.42" width="0.381" layer="156"/>
 </plain>
 <moduleinsts>
@@
 <attribute name="NAME" x="121.92" y="39.37" size="2.032" layer="95" align="bottom-center"/>
 </moduleinst>
-<moduleinst name="ENERGY_METER_BOX" module="FSAE_ENERGY_METER" x="177.8" y="127"/>
 </moduleinsts>
 <instances>
 <instance part="AIR2" gate="1" x="190.5" y="48.26" rot="R90"/>
-<instance part="AIR1" gate="1" x="340.36" y="48.26" rot="R90"/>
+<instance part="AIR1" gate="1" x="347.98" y="48.26" rot="R90"/>
 <instance part="SMD3" gate="1" x="226.06" y="48.26" rot="R90"/>
 <instance part="SMD2" gate="1" x="259.08" y="48.26" rot="R90"/>
@@
 <instance part="SEGMENT1" gate="G$1" x="322.58" y="58.42" rot="R180"/>
 <instance part="FUSE" gate="G$1" x="274.32" y="58.42"/>
-<instance part="GND5" gate="1" x="332.74" y="48.26" rot="R270"/>
+<instance part="GND5" gate="1" x="340.36" y="48.26" rot="R270"/>
 <instance part="MOLEX_IMPERIUM1" gate="G$1" x="215.9" y="116.84" rot="MR90"/>
 <instance part="U$2" gate="G$1" x="142.24" y="109.22" rot="MR0"/>
@@
 <instance part="DISCHARGE" gate="G$1" x="40.64" y="91.44"/>
 <instance part="SL2" gate="G$1" x="5.08" y="48.26" rot="MR180"/>
-<instance part="SL3" gate="G$1" x="177.8" y="104.14" rot="R90"/>
 <instance part="HVD_INTERLOCK" gate="SPST" x="256.54" y="114.3" rot="R270"/>
+<instance part="HVD" gate="G$1" x="330.2" y="53.34" rot="R90"/>
 </instances>
 <busses>
@@
 <wire x1="231.14" y1="88.9" x2="276.86" y2="88.9" width="0.1524" layer="91"/>
 <wire x1="276.86" y1="88.9" x2="276.86" y2="111.76" width="0.1524" layer="91"/>
-<wire x1="276.86" y1="111.76" x2="355.6" y2="111.76" width="0.1524" layer="91"/>
-<wire x1="355.6" y1="111.76" x2="355.6" y2="12.7" width="0.1524" layer="91"/>
+<wire x1="276.86" y1="111.76" x2="358.14" y2="111.76" width="0.1524" layer="91"/>
+<wire x1="358.14" y1="111.76" x2="358.14" y2="12.7" width="0.1524" layer="91"/>
 <label x="281.94" y="111.76" size="1.778" layer="95"/>
-<wire x1="355.6" y1="12.7" x2="96.52" y2="12.7" width="0.1524" layer="91"/>
+<wire x1="358.14" y1="12.7" x2="96.52" y2="12.7" width="0.1524" layer="91"/>
 <wire x1="96.52" y1="12.7" x2="96.52" y2="40.64" width="0.1524" layer="91"/>
 <portref moduleinst="HV_PCB" port="SHUTDOWN7_IN"/>
@@
 <wire x1="99.06" y1="15.24" x2="99.06" y2="40.64" width="0.1524" layer="91"/>
 <pinref part="AIR1" gate="1" pin="2"/>
-<wire x1="345.44" y1="30.48" x2="345.44" y2="48.26" width="0.1524" layer="91"/>
+<wire x1="353.06" y1="30.48" x2="353.06" y2="48.26" width="0.1524" layer="91"/>
 <pinref part="SMD1" gate="1" pin="2"/>
 <wire x1="309.88" y1="30.48" x2="309.88" y2="48.26" width="0.1524" layer="91"/>
-<wire x1="309.88" y1="30.48" x2="345.44" y2="30.48" width="0.1524" layer="91"/>
+<wire x1="309.88" y1="30.48" x2="353.06" y2="30.48" width="0.1524" layer="91"/>
 <junction x="309.88" y="30.48"/>
 <pinref part="SMD2" gate="1" pin="2"/>
@@
 <net name="SHUTDOWN_CIRCUIT_PRE_INTERLOCK" class="0">
 <segment>
-<wire x1="93.98" y1="10.16" x2="358.14" y2="10.16" width="0.1524" layer="91"/>
-<wire x1="358.14" y1="10.16" x2="358.14" y2="114.3" width="0.1524" layer="91"/>
+<wire x1="93.98" y1="10.16" x2="360.68" y2="10.16" width="0.1524" layer="91"/>
+<wire x1="360.68" y1="10.16" x2="360.68" y2="114.3" width="0.1524" layer="91"/>
 <label x="116.84" y="10.16" size="1.778" layer="95"/>
 <wire x1="93.98" y1="10.16" x2="93.98" y2="40.64" width="0.1524" layer="91"/>
@@
 <wire x1="261.62" y1="111.76" x2="264.16" y2="111.76" width="0.1524" layer="91"/>
 <wire x1="264.16" y1="111.76" x2="264.16" y2="114.3" width="0.1524" layer="91"/>
-<wire x1="264.16" y1="114.3" x2="358.14" y2="114.3" width="0.1524" layer="91"/>
+<wire x1="264.16" y1="114.3" x2="360.68" y2="114.3" width="0.1524" layer="91"/>
 <label x="281.94" y="114.3" size="1.778" layer="95"/>
 </segment>
@@
 </segment>
 </net>
-<net name="N$51" class="0">
-<segment>
-<portref moduleinst="ENERGY_METER_BOX" port="GND"/>
-<pinref part="SL3" gate="G$1" pin="1"/>
-<wire x1="180.34" y1="109.22" x2="180.34" y2="111.76" width="0.1524" layer="91"/>
-</segment>
-</net>
-<net name="N$52" class="0">
-<segment>
-<portref moduleinst="ENERGY_METER_BOX" port="12V+"/>
-<pinref part="SL3" gate="G$1" pin="2"/>
-<wire x1="177.8" y1="109.22" x2="177.8" y2="111.76" width="0.1524" layer="91"/>
-</segment>
-</net>
