File: ShutdownCircuitFH New 2018.sch (EAGLE design)
At the start: 30 parts

Commit message: Move 2017 schematics, update HV Board for FH2018 rules, update external diagram and wiring harness for new SSOK lamps, update FH shutdown circuit
Parts:
- removed BMS_RELAY_DRIVE, BMS_SOFTWARE_LATCH: Normally Open, HyTechDevices:SOLID_STATE_RELAY_VO14642AT
- removed HV_FUSE: (no value), HyTechSymbols:FUSE
- removed PWR: Molex Imperium, HyTechSymbols:M02
- added AMS_RELAY_DRIVE, AMS_SOFTWARE_LATCH: Normally Open, HyTechDevices:SOLID_STATE_RELAY_VO14642AT
- added FUSE: 200A, HyTechSymbols:FUSE
- added MAIN: Molex Imperium, HyTechSymbols:M02
- added SEGMENT3, SEGMENT4: BATTERY_1_CELL, HyTechSymbols:BATTERY_1_CELL
- added SMD2, SMD3: EV200, HyTechSymbols:RELAY
- added TSAL: LED, HyTechSymbols:LED
- HVD: value Hirose -> EM30MSD
Connections:
- removed net N$10: BOTS.O, INERTIA.P
- removed net N$11 (its old number): INERTIA.O, SOFTWARE_SHUTOFF.P
- removed net N$15: U$3.CTCS-
- new net N$14: TSAL.A
- new net N$17: BOTS.P, INERTIA.O
- new net TO_GLV_SYSTEMS: LEFT_BRB.O, U$1.6
- new net TO_SSOK_LAMPS: BOTS.O, COCKPIT_BRB.P
- net GND: now also AMS_RELAY_DRIVE.LED-, AMS_SOFTWARE_LATCH.LED-, SMD2.2, SMD3.2, TSAL.C; no longer BMS_RELAY_DRIVE.LED-, BMS_SOFTWARE_LATCH.LED-
- net ISO+: now also U$3.CTCS-
- net ISO-: now also MAIN.2; no longer PWR.2
- net N$13: now also AMS_RELAY_DRIVE.IO2, AMS_SOFTWARE_LATCH.IO1; no longer BMS_RELAY_DRIVE.IO2, BMS_SOFTWARE_LATCH.IO1
- net N$16: now also AMS_SOFTWARE_LATCH.IO2; no longer BMS_SOFTWARE_LATCH.IO2
- net N$8: now also INERTIA.P; no longer COCKPIT_BRB.P
- net N$9: now also SOFTWARE_SHUTOFF.P; no longer BOTS.P
- net SHUTDOWN_CIRCUIT: now also SMD2.1, SMD3.1
- net VIN: now also AMS_RELAY_DRIVE.IO1, AMS_RELAY_DRIVE.LED+, AMS_SOFTWARE_LATCH.LED+; no longer BMS_RELAY_DRIVE.IO1, BMS_RELAY_DRIVE.LED+, BMS_SOFTWARE_LATCH.LED+, LEFT_BRB.O, U$1.6
Other:
- note added: "AMS OK signal"
- note added: "TODO: Changing Latching Mechanism"
- note removed: "BMS OK signal"
- note removed: "HV_ISO+"
- note removed: "HV_ISO-"
- note removed: "To GLV Systems"
- moved on the sheet: AIR1, AIR2, BSPD, COCKPIT_BRB, FUSE1, FUSE2, GLVMS, GLV_BATTERY, HVD, INERTIA, LEFT_BRB, RIGHT_BRB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

Commit message: Update shutdown circuit for FH ESF
Parts:
- renumbered AMS_SOFTWARE_LATCH to AMS_STATE_LATCH, IMD_SOFTWARE_LATCH to IMD_STATE_LATCH
Other:
- note added: "State machine signal"
- note removed: "Software latch signal"
- note removed: "TODO: Changing Latching Mechanism"
Changed lines of the file:
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@@
 <part name="LEFT_BRB" library="HyTechSymbols" deviceset="SWITCH_SPST" device="" value="Normally Closed"/>
 <part name="U$1" library="HyTechDevices" deviceset="G2RL-2-DC12" device=""/>
-<part name="AMS_SOFTWARE_LATCH" library="HyTechDevices" deviceset="SOLID_STATE_RELAY" device="_VO14642AT" value="Normally Open"/>
+<part name="AMS_STATE_LATCH" library="HyTechDevices" deviceset="SOLID_STATE_RELAY" device="_VO14642AT" value="Normally Open"/>
 <part name="AMS_RELAY_DRIVE" library="HyTechDevices" deviceset="SOLID_STATE_RELAY" device="_VO14642AT" value="Normally Open"/>
-<part name="IMD_SOFTWARE_LATCH" library="HyTechDevices" deviceset="SOLID_STATE_RELAY" device="_VO14642AT" value="Normally Open"/>
+<part name="IMD_STATE_LATCH" library="HyTechDevices" deviceset="SOLID_STATE_RELAY" device="_VO14642AT" value="Normally Open"/>
 <part name="U$2" library="HyTechSymbols" deviceset="BENDER_IR155-3204" device=""/>
 <part name="GND2" library="HyTechSymbols" deviceset="GND" device=""/>
@@
 <text x="116.84" y="48.26" size="1.778" layer="97" rot="R180">Insulation Monitoring Device</text>
 <text x="149.86" y="102.87" size="1.778" layer="95" rot="MR180" align="top-left">AMS OK signal</text>
-<text x="149.86" y="125.73" size="1.778" layer="95" rot="MR180" align="top-left">Software latch signal</text>
-<text x="129.54" y="151.13" size="1.778" layer="95" rot="MR180" align="top-left">Software latch signal</text>
-<text x="68.58" y="162.56" size="5.08" layer="91">TODO: Changing Latching Mechanism</text>
+<text x="149.86" y="125.73" size="1.778" layer="95" rot="MR180" align="top-left">State machine signal</text>
+<text x="129.54" y="151.13" size="1.778" layer="95" rot="MR180" align="top-left">State machine signal</text>
 <wire x1="10.16" y1="20.32" x2="7.62" y2="20.32" width="0.6096" layer="156"/>
 <wire x1="7.62" y1="20.32" x2="7.62" y2="7.62" width="0.6096" layer="156"/>
@@
 <instance part="LEFT_BRB" gate="SPST" x="63.5" y="111.76" rot="R270"/>
 <instance part="U$1" gate="G$1" x="83.82" y="134.62" rot="R270"/>
-<instance part="AMS_SOFTWARE_LATCH" gate="G$1" x="139.7" y="127" rot="R180"/>
+<instance part="AMS_STATE_LATCH" gate="G$1" x="139.7" y="127" rot="R180"/>
 <instance part="AMS_RELAY_DRIVE" gate="G$1" x="139.7" y="104.14" rot="R180"/>
-<instance part="IMD_SOFTWARE_LATCH" gate="G$1" x="119.38" y="152.4" rot="R180"/>
+<instance part="IMD_STATE_LATCH" gate="G$1" x="119.38" y="152.4" rot="R180"/>
 <instance part="U$2" gate="G$1" x="132.08" y="73.66" rot="R180"/>
 <instance part="GND2" gate="1" x="73.66" y="50.8" rot="R270"/>
@@
 </segment>
 <segment>
-<pinref part="AMS_SOFTWARE_LATCH" gate="G$1" pin="LED-"/>
+<pinref part="AMS_STATE_LATCH" gate="G$1" pin="LED-"/>
 <pinref part="GND5" gate="1" pin="GND"/>
 <wire x1="152.4" y1="129.54" x2="149.86" y2="129.54" width="0.1524" layer="91"/>
 </segment>
 <segment>
-<pinref part="IMD_SOFTWARE_LATCH" gate="G$1" pin="LED-"/>
+<pinref part="IMD_STATE_LATCH" gate="G$1" pin="LED-"/>
 <pinref part="GND6" gate="1" pin="GND"/>
 <wire x1="132.08" y1="154.94" x2="129.54" y2="154.94" width="0.1524" layer="91"/>
@@
 <segment>
 <pinref part="LATCH_SIGNAL" gate="G$1" pin="VIN"/>
-<pinref part="IMD_SOFTWARE_LATCH" gate="G$1" pin="LED+"/>
+<pinref part="IMD_STATE_LATCH" gate="G$1" pin="LED+"/>
 <wire x1="132.08" y1="149.86" x2="129.54" y2="149.86" width="0.1524" layer="91"/>
 </segment>
 <segment>
 <pinref part="SOFTWARE_OK_SIGNAL" gate="G$1" pin="VIN"/>
-<pinref part="AMS_SOFTWARE_LATCH" gate="G$1" pin="LED+"/>
+<pinref part="AMS_STATE_LATCH" gate="G$1" pin="LED+"/>
 <wire x1="152.4" y1="124.46" x2="149.86" y2="124.46" width="0.1524" layer="91"/>
 </segment>
@@
 <net name="N$13" class="0">
 <segment>
-<pinref part="AMS_SOFTWARE_LATCH" gate="G$1" pin="IO1"/>
+<pinref part="AMS_STATE_LATCH" gate="G$1" pin="IO1"/>
 <wire x1="129.54" y1="124.46" x2="116.84" y2="124.46" width="0.1524" layer="91"/>
 <wire x1="116.84" y1="124.46" x2="116.84" y2="114.3" width="0.1524" layer="91"/>
@@
 <wire x1="76.2" y1="154.94" x2="76.2" y2="129.54" width="0.1524" layer="91"/>
 <junction x="76.2" y="129.54"/>
-<pinref part="IMD_SOFTWARE_LATCH" gate="G$1" pin="IO2"/>
+<pinref part="IMD_STATE_LATCH" gate="G$1" pin="IO2"/>
 </segment>
 </net>
@@
 <wire x1="99.06" y1="137.16" x2="124.46" y2="137.16" width="0.1524" layer="91"/>
 <wire x1="124.46" y1="137.16" x2="124.46" y2="129.54" width="0.1524" layer="91"/>
-<pinref part="AMS_SOFTWARE_LATCH" gate="G$1" pin="IO2"/>
+<pinref part="AMS_STATE_LATCH" gate="G$1" pin="IO2"/>
 <wire x1="124.46" y1="129.54" x2="129.54" y2="129.54" width="0.1524" layer="91"/>
 <pinref part="U$4" gate="G$1" pin="3"/>
@@
 <wire x1="96.52" y1="116.84" x2="93.98" y2="116.84" width="0.1524" layer="91"/>
 <wire x1="96.52" y1="149.86" x2="96.52" y2="140.97" width="0.1524" layer="91"/>
-<pinref part="IMD_SOFTWARE_LATCH" gate="G$1" pin="IO1"/>
+<pinref part="IMD_STATE_LATCH" gate="G$1" pin="IO1"/>
 <wire x1="96.52" y1="140.97" x2="96.52" y2="116.84" width="0.1524" layer="91"/>
 <wire x1="109.22" y1="149.86" x2="96.52" y2="149.86" width="0.1524" layer="91"/>
