File: 2017 Schematics/External Diagram 2017.sch (EAGLE design)
At the start: 84 parts

Commit message: Move old schematics, update 2018 diagram to 4 segments, Rules-compliant resistors, and add AMS test port
Parts:
- removed SEGMENT3, SEGMENT4: BATTERY_1_CELL, HyTechSymbols:BATTERY_1_CELL
- removed SL1: (no value), HyTechSymbols:M12
- removed SL13: (no value), HyTechSymbols:M02
- removed SMD2, SMD3: GX23BA, HyTechSymbols:RELAY
- removed TSMP_RES+_1, TSMP_RES+_2, TSMP_RES-_1, TSMP_RES-_2: 5k, HyTechDevices:RESISTOR10W
- added SL24, SL25: (no value), HyTechSymbols:M08
- added SL28: (no value), HyTechSymbols:M02
- added TSMP_RES+, TSMP_RES-: 5k, HyTechDevices:RESISTOR10W
- SL5: device HyTechSymbols:M10 -> HyTechSymbols:M02
- SL7: device HyTechSymbols:M10 -> HyTechSymbols:M08
- SL9: device HyTechSymbols:M12 -> HyTechSymbols:M08
Connections:
- removed net 12VSUPPLY_BRB: SL15.1, SL5.2
- removed net FAN1-: SL8.8
- removed net FAN2-: SL8.9
- removed net GPIO_1: SL1.10, SL8.6
- removed net GPIO_2: SL1.11, SL5.9
- removed net GPIO_3: SL1.12, SL5.10
- removed net N$10: SL13.1, SL13.2
- removed net N$11: SL18.1
- removed net N$35 (its old number): SL18.2
- removed net N$41 (its old number): TSMP_RES-_1.1, TSMP_RES-_2.2
- removed net N$57: TSMP_RES+_1.1, TSMP_RES+_2.2
- removed net N$7: SL7.9
- removed net N$9: SL7.10
- removed net PUMP1-: SL8.7
- new net BUS_REAR->ACCUM_: SL4.13
- new net GPIO: SL8.6
- new net N$79: SL5.2, SL8.9
- new net N$94: SL18.2, SL8.8
- new net N$95: SL28.2, SL8.7
- new net TSAL: SL25.4, TSAL/TSEL.A
- net 12VSUPPLY: now also SL15.1, SL9.2
- net 12VSUPPLY_COOLING: now also SL18.1, SL28.1, SL5.1
- net 12VSUPPLY_COOLING_UNSWITCHED: now also SL24.2, SL25.2; no longer SL1.2, SL9.2
- net 12VSUPPLY_FSAE: now also SL24.8, SL25.8, SL9.1; no longer SL1.8, SL5.1, SL9.8
- net 12VSUPPLY_UNSWITCHED: now also SL24.1, SL25.1; no longer SL1.1, SL9.1
- net BAT+: no longer SL1.9, SL9.9
- net BUS_REAR->ACCUM_12VSUPPLY: now also SL9.4; no longer SL4.13, SL5.4
- net BUS_REAR->ACCUM_CANH: no longer SL5.8
- net BUS_REAR->ACCUM_CANL: no longer SL5.7
- net BUS_REAR->ACCUM_GND: no longer SL5.6
- net BUS_REAR->FRONT_12VSUPPLY: now also SL9.5; no longer SL5.5
- net BUS_REAR->FRONT_CANH: now also SL9.8
- net BUS_REAR->FRONT_CANL: now also SL9.7
- net BUS_REAR->FRONT_GND: now also SL9.6
- net CHARGE_ENABLE: now also SL24.7, SL25.7; no longer SL1.7, SL9.7
- net GND: now also SL9.3; no longer SL5.3, SMD2.2, SMD3.2
- net N$20: no longer TSMP_RES-_2.1
- net N$34: no longer TSMP_RES+_2.1
- net N$39: now also TSMP_RES-.2; no longer TSMP_RES-_1.2
- net N$40: now also TSMP_RES+.2; no longer TSMP_RES+_1.2
- net SHUTDOWN5: now also SL24.5, SL25.5; no longer SL1.5, SL9.5
- net SHUTDOWN6: now also SL24.6, SL25.6; no longer SL1.6, SL9.6
- net SHUTDOWN7: no longer SMD2.1, SMD3.1
- net TSAL+: now also SL24.4; no longer SL1.4, SL9.4, TSAL/TSEL.A
- net TSVP+: now also SL24.3, SL25.3; no longer SL1.3, SL9.3
Other:
- note added: "HyTech Racing 2017 Electrical Diagram"
- note removed: "HyTech Racing 2018 Electrical Diagram"
- note removed: "⬅ Disconnected for Formula Hybrid"
- note removed: "⬅ Formula Hybrid AMS Test Port"
- moved on the sheet: AIR1, AIR2, CHARGE_ENABLE, EM_F1, F3, FUSE, GLVMS, GLV_BATT, HVD, HVD_INTERLOCK, IMPERIUM_INTERLOCK, MEASURE_12V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
