File: Board Designs/Latch Manager/SMD/latch3.brd (EAGLE design)
At the start: 55.9 x 49.8 mm, 26 parts, among them IC1 SN74AHC00D, IC2 SN74AHC74D, IC3 SN74AHC00D, IC4 SN74AHC74D, IC6 SN74AHC00D, X1 CONNECTOR-4, X2 CONNECTOR-2, Y1 16MHz

Commit message: Adding latching board manager revisions
Parts:
- removed R1, R2, R4, R5: (no value), HyTechDevices:0402-RES
- moved C1 5.79 mm to (19.8, 28.3), turned to 270 degrees
- moved IC6 1.27 mm to (42.4, 20.8)
- moved R9 1.20 mm to (10.8, 15.5), turned to 90 degrees
- moved C2 1.14 mm to (30.5, 26.7)
Connections:
- removed net BMS_DEBOUNCE: C1.2, IC3.2, IC6.1, IC6.2, R4.2
- removed net IMD_DEBOUNCE: C2.2, IC1.1, IC1.2, IC1.9, R5.2
- net +5V: no longer R1.1, R2.2
- net BMS_5V: now also IC3.2, IC6.1, IC6.2; no longer R1.2, R4.1
- net GND: now also C1.2, C2.1
- net IMD_5V: now also C2.2, IC1.1, IC1.2, IC1.9; no longer C2.1, R2.1, R5.1
Routing:
- net BMS_DEBOUNCE: track 106.1 -> 0.00 mm, vias 3 -> 0
- net BMS_5V: track 6.28 -> 109.9 mm, vias 0 -> 3
- net IMD_DEBOUNCE: track 25.4 -> 0.00 mm, vias 3 -> 0
- net IMD_5V: track 7.07 -> 29.8 mm, vias 0 -> 3
- net +5V: track 222.8 -> 207.1 mm
- net GND: track 192.5 -> 201.9 mm
- net N$33: track 16.7 -> 15.0 mm
- net N$32: track 20.9 -> 19.5 mm
- net N$8: track 95.2 -> 93.9 mm
- net N$23: track 27.6 -> 28.9 mm
- net N$21: track 36.0 -> 34.7 mm
- net N$12: track 10.9 -> 12.2 mm
- net IMD_OUT: track 119.7 -> 118.4 mm
- net BMS_IN: track 2.34 -> 3.24 mm
- net N$7: track 62.3 -> 63.2 mm
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