File: Board Designs/BMS/BMS Segment/BMS Segment rev3/BMS Segment rev3.sch (EAGLE design)
At the start: 68 parts, among them T1 NPN_BCP56T1, X1 CONNECTOR-2NANO-FIT_VERTICAL-2, X2 CONNECTOR-2NANO-FIT_VERTICAL-2, X3 Th1, X4 Th2, X5 Th3

Commit message: BMS Rev3 Schematic
Added new BMS rev3 schematic
Parts:
- removed C6, C7: 25pF, HyTechDevices:CAP0805
- removed CR0, CR1, CR10, CR2, CR3, CR4, CR5, CR7, CR8, CR9: 10nF, HyTechDevices:CAP0805
- removed R1, R49: 120Ω, HyTechDevices:RESISTOR0805-RES
- removed R101, R102, R103: 10kΩ, HyTechDevices:RESISTOR0805-RES
- removed RC0, RC1, RC10, RC2, RC3, RC4, RC5, RC7, RC8, RC9, S2: 100Ω, HyTechDevices:RESISTOR0805-RES
- removed SC1: 0.1uF, HyTechDevices:CAP0805
- removed T1: NPN_BCP56T1, HyTechDevices:NPN_BCP56T1
- removed TEST_PORT: MINIFIT_5566-4, HyTechDevices:MINIFIT_5566-4
- removed TO_TOP, X2: CONNECTOR-2NANO-FIT_VERTICAL-2, HyTechDevices:CONNECTOR-2NANO-FIT_VERTICAL-2
- removed TRANSFORMER-: 350uH, HyTechDevices:TRANSFORMER_749010013
- added ADP2360: ADP2360, HyTechDevices:ADP2360
- added AMS_TEST_PORT: CONNECTOR-2NANO-FIT_VERTICAL-2, HyTechDevices:CONNECTOR-2NANO-FIT_VERTICAL-2
- added C, C4: 10nF, HyTechDevices:CAP0805
- added CIN: 4.7uF, HyTechDevices:CAP0805
- added COUT: 22uF, HyTechDevices:CAP0805
- added CSS: 2.2nF, HyTechDevices:CAP0805
- added J1, J2, J3, J4, J5, J6, J7, J8, J9: (no value), HyTechDevices:RESISTOR0805-RES
- added L1: 330uH, HyTechDevices:SRU1048
- added R, RM: 100Ω, HyTechDevices:RESISTOR0805-RES
- added R6, R7: 22Ω, HyTechDevices:RESISTOR0805-RES
- added R8: 402Ω, HyTechDevices:RESISTOR0805-RES
- added R9, RPG: 1kΩ, HyTechDevices:RESISTOR0805-RES
- added THERM1, THERM2: 10kΩ, HyTechDevices:THERMISTOR_NCP210603
- added TRANSFORMER: SM51589PEL, HyTechDevices:SM51589PEL
- C3: value 1uF -> 15pF
- F0, F1, F2, F3, F4, F5, F6, F7, F8, F9: value 0751.0110_FUSE_CLIP -> 0001.2704.11; device HyTechDevices:0751.0110_FUSE_CLIP -> HyTechDevices:0001.2704.11
- RB2: value 1.2kΩ -> 800Ω
- U$2: value (none) -> LTC6804-2; device HyTechDevices:LTC6804-1 -> HyTechDevices:LTC6804-2
Connections:
- removed net ISOSPI-M_IN: TRANSFORMER-R.D-, X1-2.S
- removed net ISOSPI-M_OUT: TRANSFORMER-T.D-, X2-2.S
- removed net ISOSPI-P_IN: TRANSFORMER-R.D+, X1-1.S
- removed net ISOSPI-P_OUT: TRANSFORMER-T.D+, X2-1.S
- removed net N$42: R1.2, TRANSFORMER-T.X-, U$2.IMB
- removed net SENSE1_J: RC1.1, TEST_PORT-4.S
- removed net SUPPLY: S1.2, SC1.1, T1.COLLECTOR
- removed net THERMISTOR1: R101.2, U$2.GPI01, X5-2.S
- removed net THERMISTOR2: R102.2, U$2.GPI02, X4-2.S
- removed net THERMISTOR3: R103.2, U$2.GPI03, X3-2.S
- new net C(N): C.1, R.2
- new net CELL+: R.1
- new net GPIO: C1.1
- new net GPIO1: U$2.GPI01
- new net GPIO2: U$2.GPI02
- new net GPIO3: U$2.GPI03
- new net GPIO4: U$2.GPI04
- new net GPIO5: U$2.GPI05
- new net IM: C3.2, TRANSFORMERG$1.TD+, U$2.CSB(IMA)
- new net IP: R8.1, TRANSFORMERG$1.TD-, U$2.SCK(IPA)
- new net ISOSPI-M: R7.2, RM.2, X1-2.S
- new net ISOSPI-P: R6.2, RM.1, X1-1.S
- new net N$10: C3.1, R8.2
- new net N$11: ADP2360.VIN, CIN.1, R9.2, RPG.2
- new net N$12: ADP2360.PG, RPG.1
- new net N$13: J3.1, J4.1, U$2.A1
- new net N$14: ADP2360.SS, CSS.2
- new net N$15: ADP2360.SW, L1.P$1
- new net N$16: J1.1, J2.1, U$2.A0
- new net N$17: THERM2.2
- new net N$18: X4-2.S
- new net N$19: THERM1.2
- new net N$26: X5-2.S
- new net N$3: X3-2.S
- new net SENSE9_J: AMS_TEST_PORT-1.S, F9.2, J9.1
- net C0: now also C.1, R.2; no longer CR0.1, CR1.2, RC0.2
- net C1: no longer CR1.1, CR2.2, RC1.2
- net C10: no longer CR10.1, RC10.2
- net C2: no longer CR2.1, CR3.2, RC2.2
- net C3: no longer CR3.1, CR4.2, RC3.2
- net C4: no longer CR4.1, CR5.2, RC4.2
- net C5: no longer CR5.1, CR7.2, RC5.2
- net C7: no longer CR7.1, CR8.2, RC7.2
- net C8: no longer CR8.1, CR9.2, RC8.2
- net C9: no longer CR10.2, CR9.1, RC9.2
- net DRIVE: now also ADP2360.EN; no longer T1.BASE
- net N$1: now also C4.1, TRANSFORMERG$1.TCT; no longer C7.1, TRANSFORMER-R.CX
- net N$2: now also RB1.2, U$2.SDO(IBIAS); no longer C6.1, TRANSFORMER-T.CX
- net N$4: now also RB1.1, RB2.2, U$2.SDI(ICMP); no longer RB1.2, U$2.IBIAS
- net N$5: now also R6.1, TRANSFORMERG$1.MX-; no longer R1.1, TRANSFORMER-T.X+, U$2.IPB
- net N$7: now also R7.1, TRANSFORMERG$1.MX+; no longer RB1.1, RB2.2, U$2.ICMP
- net N$8: now also J7.1, J8.1, U$2.A3; no longer R49.1, TRANSFORMER-R.X+, U$2.SCK(IPA)
- net N$9: now also J5.1, J6.1, U$2.A2; no longer R49.2, TRANSFORMER-R.X-, U$2.CSB(IMA)
- net SENSE1: no longer TEST_PORT-2.S
- net SENSE2: no longer RC2.1
- net SENSE3: no longer RC3.1
- net SENSE4: no longer RC4.1
- net SENSE5: no longer RC5.1
- net SENSE6: no longer RC7.1
- net SENSE7: no longer RC8.1
- net SENSE8: no longer RC9.1
- net SENSE9: now also AMS_TEST_PORT-2.S, J9.2; no longer F9.2, RC10.1, S2.1, TO_TOP-1.S, TO_TOP-2.S
- net V+: now also R9.1, S1.2; no longer S2.2
- net V-: now also ADP2360.AGND, ADP2360.ITH, ADP2360.PGND, C.2, C4.2, CIN.2, COUT.1, CSS.1, J1.2, J3.2, J5.2, J7.2, R.1, THERM1.1, THERM2.1; no longer C3.2, C6.2, C7.2, CR0.2, RC0.1, SC1.2, TEST_PORT-3.S, U$2.SDI(NC), U$2.SDO(NC)
- net VREF2: no longer R101.1, R102.1, R103.1
- net VREG: now also ADP2360.FB, COUT.2, J2.2, J4.2, J6.2, J8.2, L1.P$2; no longer C3.1, T1.EMITTER
Other:
- note added: "3 cell thermistors and 2 PCB thermistors per LTC6804 IC"
- note added: "Cell Input"
- note added: "RM is only to be connected on LAST segment"
- note added: "See LTC6804 DATASHEET pg.61"
- note added: "ceramic / 40+V"
- note removed: "ISOMD connected to VREG enables 2-wire isoSPI mode"
- note removed: "SWTEN connected to VREG enables Software Timer"
- note removed: "See LTC6804-1 DATASHEET pg.61"
- note removed: "TODO: Calculate RB1 and RB2 Verify Enable Pins"
- note removed: "Total of 6 termistors per 18 cell segment"
- moved on the sheet: C1, C2, C3, CELL0, CELL1, CELL2, CELL3, CELL4, CELL5, CELL6, CELL7, CELL8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

Commit message: BMS Finished Schematic and Preliminary Board
Completed BMS schematic layout for 18 cell BMS segment board.  Finished a preliminary component layout for the board design, but no traces have been routed yet.
Parts:
- removed AMS_TEST_PORT: CONNECTOR-2NANO-FIT_VERTICAL-2, HyTechDevices:CONNECTOR-2NANO-FIT_VERTICAL-2
- removed C: 10nF, HyTechDevices:CAP0805
- removed C1: 1uF, HyTechDevices:CAP0805
- removed CIN: 4.7uF, HyTechDevices:CAP0805
- removed J9: (no value), HyTechDevices:RESISTOR0805-RES
- removed R: 100Ω, HyTechDevices:RESISTOR0805-RES
- added AMS_TEST_PORT1, ISOSPI_A: CONNECTOR-2NANO-FIT_VERTICAL-2, HyTechDevices:CONNECTOR-2NANO-FIT_VERTICAL-2
- added BUCK_CONV_A: ADP2360, HyTechDevices:ADP2360
- added C1_A, C1_B, C2_A: 1uF, HyTechDevices:CAP0805
- added C3_A: 15pF, HyTechDevices:CAP0805
- added C4_A, C5_A, C_5: 10nF, HyTechDevices:CAP0805
- added C6_A: 0.1uF, HyTechDevices:CAP0805
- added CELL10, CELL11, CELL12, CELL13, CELL14, CELL15, CELL16, CELL17, CELL18: BATTERY_SPRING_KEYSTONE5222, HyTechDevices:BATTERY_SPRING_KEYSTONE5222
- added CIN_A, CIN_B: 4.7uF, HyTechDevices:CAP0805
- added COUT_A: 22uF, HyTechDevices:CAP0805
- added CSS_A: 2.2nF, HyTechDevices:CAP0805
- added F10, F11, F12, F13, F14, F15, F16, F17, F18: 0001.2704.11, HyTechDevices:0001.2704.11
- added J, J1_A, J2_A, J3_A, J4_A, J5_A, J6_A, J7_A, J8_A: (no value), HyTechDevices:RESISTOR0805-RES
- added L1_A: 330uH, HyTechDevices:SRU1048
- added R1_A, R2_A, R2_B, RM_A, RU1_A, RU2_A: 100Ω, HyTechDevices:RESISTOR0805-RES
- added R3_A: 402Ω, HyTechDevices:RESISTOR0805-RES
- added R4_A, R5_A: 22Ω, HyTechDevices:RESISTOR0805-RES
- added RB1_A: 1.2kΩ, HyTechDevices:RESISTOR0805-RES
- added RB2_A: 800Ω, HyTechDevices:RESISTOR0805-RES
- added RIN_A, RPG_A: 1kΩ, HyTechDevices:RESISTOR0805-RES
- added THERM1A: Th1, HyTechDevices:CONNECTOR-2NANO-FIT_VERTICAL-2
- added THERM2A: Th2, HyTechDevices:CONNECTOR-2NANO-FIT_VERTICAL-2
- added THERM3, THERM4: 10kΩ, HyTechDevices:THERMISTOR_NCP210603
- added THERM3A: Th3, HyTechDevices:CONNECTOR-2NANO-FIT_VERTICAL-2
- added U$1: LTC6804-2, HyTechDevices:LTC6804-2
- renumbered ADP2360 to BUCK_CONV_B, C2 to C2_B, C3 to C3_B, C4 to C4_B, COUT to COUT_B, CSS to CSS_B, J1 to J1_B, J2 to J2_B, J3 to J3_B, J4 to J4_B, J5 to J5_B, J6 to J6_B, J7 to J7_B, J8 to J8_B, L1 to L1_B, R6 to R4_B, R7 to R5_B, R8 to R3_B, R9 to RIN_B, RB1 to RB1_B, RB2 to RB2_B, RM to RM_B, RPG to RPG_B, RU1 to RU1_B, RU2 to RU2_B, S1 to R1_B, SC2 to C6_B, X1 to ISOSPI_B, X3 to THERM1_B, X4 to THERM2_B, X5 to THERM3_B
Connections:
- net C1 renamed C1_B
- net C10 renamed C10_B
- net C2 renamed C2_B
- net C3 renamed C3_B
- net C4 renamed C4_B
- net C5 renamed C5_B
- net C7 renamed C7_B
- net C8 renamed C8_B
- net C9 renamed C9_B
- net DRIVE renamed DRIVE_B
- net GPIO1 renamed GPIO1_B
- net GPIO2 renamed GPIO2_B
- net GPIO3 renamed GPIO3_B
- net GPIO4 renamed GPIO4_B
- net GPIO5 renamed GPIO5_B
- net IM renamed IM_B
- net IP renamed IP_B
- net ISOSPI-M renamed ISOSPI-M_B
- net ISOSPI-P renamed ISOSPI-P_B
- net S1 renamed S1_B
- net S10 renamed S10_B
- net S2 renamed S2_B
- net S3 renamed S3_B
- net S4 renamed S4_B
- net S5 renamed S5_B
- net S7 renamed S7_B
- net S8 renamed S8_B
- net S9 renamed S9_B
- net UNUSED1 renamed UNUSED1_B
- net UNUSED2 renamed UNUSED2_B
- net V+ renamed V+_B
- net VREF1 renamed VREF1_B
- net VREG renamed VREG_B
- removed net C(N): C.1, R.2
- removed net C0: C.1, R.2, U$2.C0
- removed net CELL+: R.1
- removed net GPIO: C1.1
- removed net SENSE9: AMS_TEST_PORT-2.S, J9.2, R1_B.1, RU1_B.1
- removed net SENSE9_J: AMS_TEST_PORT-1.S, F9.2, J9.1
- removed net V-: BUCK_CONV_B.AGND, BUCK_CONV_B.ITH, BUCK_CONV_B.PGND, C.2, C1.2, C2_B.2, C4_B.2, C6_B.2, CIN.2, COUT_B.1, CSS_B.1, F0.2, J1_B.2, J3_B.2, J5_B.2, J7_B.2, R.1, RB2_B.1, THERM1.1, THERM1_B-1.S, THERM2.1, THERM2_B-1.S, THERM3_B-1.S, U$2.V-, U$2.V-**
- removed net VREF2: C1.1, U$2.VREF2
- new net C0_A: C5_A.1, R2_A.2, U$1.C0
- new net C0_B: C_5.1, R2_B.2, U$2.C0
- new net C10_A: U$1.C10
- new net C1_A: U$1.C1
- new net C2_A: U$1.C2
- new net C3_A: U$1.C3
- new net C4_A: U$1.C4
- new net C5_A: U$1.C5
- new net C7_A: U$1.C7
- new net C8_A: U$1.C8
- new net C9_A: U$1.C9
- new net CC10: CELL10.S, F10.1
- new net CC11: CELL11.S, F11.1
- new net CC12: CELL12.S, F12.1
- new net CC13: CELL13.S, F13.1
- new net CC14: CELL14.S, F14.1
- new net CC15: CELL15.S, F15.1
- new net CC16: CELL16.S, F16.1
- new net CC17: CELL17.S, F17.1
- new net CC18: CELL18.S, F18.1
- new net DRIVE_A: BUCK_CONV_A.EN, U$1.DRIVE
- new net GPIO1_A: U$1.GPI01
- new net GPIO2_A: U$1.GPI02
- new net GPIO3_A: U$1.GPI03
- new net GPIO4_A: U$1.GPI04
- new net GPIO5_A: U$1.GPI05
- new net IM_A: C3_A.2, TRANSFORMERG$2.TD+, U$1.CSB(IMA)
- new net IP_A: R3_A.1, TRANSFORMERG$2.TD-, U$1.SCK(IPA)
- new net ISOSPI-M_A: ISOSPI_A-2.S, R5_A.2, RM_A.2
- new net ISOSPI-P_A: ISOSPI_A-1.S, R4_A.2, RM_A.1
- new net N$17: THERM4.2
- new net N$19: THERM3.2
- new net N$20: RB1_A.1, RB2_A.2, U$1.SDI(ICMP)
- new net N$21: C4_A.1, TRANSFORMERG$2.TCT
- new net N$22: R4_A.1, TRANSFORMERG$2.MX-
- new net N$23: R5_A.1, TRANSFORMERG$2.MX+
- new net N$24: C3_A.1, R3_A.2
- new net N$25: BUCK_CONV_A.VIN, CIN_A.1, RIN_A.2, RPG_A.2
- new net N$27: BUCK_CONV_A.PG, RPG_A.1
- new net N$28: BUCK_CONV_A.SS, CSS_A.2
- new net N$29: BUCK_CONV_A.SW, L1_A.P$1
- new net N$30: J7_A.1, J8_A.1, U$1.A3
- new net N$31: J5_A.1, J6_A.1, U$1.A2
- new net N$32: J3_A.1, J4_A.1, U$1.A1
- new net N$33: J1_A.1, J2_A.1, U$1.A0
- new net N$35: THERM3A-2.S
- new net N$37: THERM2A-2.S
- new net N$38: THERM1A-2.S
- new net N$6: RB1_A.2, U$1.SDO(IBIAS)
- new net S10_A: U$1.S10
- new net S1_A: U$1.S1
- new net S2_A: U$1.S2
- new net S3_A: U$1.S3
- new net S4_A: U$1.S4
- new net S5_A: U$1.S5
- new net S7_A: U$1.S7
- new net S8_A: U$1.S8
- new net S9_A: U$1.S9
- new net SENSE10: F10.2
- new net SENSE11: F11.2
- new net SENSE12: F12.2
- new net SENSE13: F13.2
- new net SENSE14: F14.2, RU2_A.1
- new net SENSE15: F15.2
- new net SENSE16: F16.2
- new net SENSE17: F17.2
- new net SENSE18: AMS_TEST_PORT1-2.S, J.2, R1_A.1, RU1_A.1
- new net SENSE18_J: AMS_TEST_PORT1-1.S, F18.2, J.1
- new net UNUSED1_A: RU1_A.2, U$1.C11, U$1.C12
- new net UNUSED2_A: RU2_A.2, U$1.C6
- new net V+_A: C6_A.1, R1_A.2, RIN_A.1, U$1.V+
- new net V-_A: BUCK_CONV_A.AGND, BUCK_CONV_A.ITH, BUCK_CONV_A.PGND, C1_A.2, C2_A.2, C4_A.2, C5_A.2, C6_A.2, CIN_A.2, COUT_A.1, CSS_A.1, F9.2, J1_A.2, J3_A.2, J5_A.2, J7_A.2, R1_B.1, R2_A.1, RB2_A.1, RU1_B.1, THERM1.1, THERM1A-1.S, THERM2.1, THERM2A-1.S, THERM3A-1.S, U$1.V-, U$1.V-**
- new net V-_B: BUCK_CONV_B.AGND, BUCK_CONV_B.ITH, BUCK_CONV_B.PGND, C1_B.2, C2_B.2, C4_B.2, C6_B.2, CIN_B.2, COUT_B.1, CSS_B.1, C_5.2, F0.2, J1_B.2, J3_B.2, J5_B.2, J7_B.2, R2_B.1, RB2_B.1, THERM1_B-1.S, THERM2_B-1.S, THERM3.1, THERM3_B-1.S, THERM4.1, U$2.V-, U$2.V-**
- new net VREF1_A: C2_A.1, U$1.VREF1
- new net VREF2_A: C1_A.1, U$1.VREF2
- new net VREF2_B: C1_B.1, U$2.VREF2
- new net VREG_A: BUCK_CONV_A.FB, COUT_A.2, J2_A.2, J4_A.2, J6_A.2, J8_A.2, L1_A.P$2, U$1.ISOMD, U$1.SWTEN, U$1.VREG
- net N$11: now also CIN_B.1; no longer CIN.1
Other:
- note added: "CELL 9 IS SHARED BY CIRCUIT A AND CIRCUIT B"
- note added: "Circuit A (Upper 9 Cells)"
- note added: "Circuit B (Lower 9 Cells)"
- note added: "SENSE9"
- note added: "V-_A / SENSE9"
- moved on the sheet: CELL9, F9, THERM1, THERM2, TRANSFORMERG$2

Commit message: Completed BMS Segment Board
Completed both schematic and board for BMS segments.  Ready for manufacturing pending approval from Linear's applications engineer(s)
Other:
- note added: "0Ω jumper resistors to set chip address"
- note added: "ADP2360"
- note added: "LTC6804-2"
Changed lines of the file:
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@@
 <?xml version="1.0" encoding="utf-8"?>
 <!DOCTYPE eagle SYSTEM "eagle.dtd">
-<eagle version="8.4.0">
+<eagle version="8.4.1">
 <drawing>
 <settings>
@@
 </variantdefs>
 <parts>
-<part name="GATE1" library="HyTechDevices" deviceset="RESISTOR" device="0805-RES" value="3.3kΩ"/>
-<part name="W1" library="HyTechDevices" deviceset="RESISTOR" device="PWR163" value="5Ω"/>
-<part name="PFET1" library="HyTechDevices" deviceset="P-CHANNEL_MOSFET_DMP3099L-7" device=""/>
+<part name="GATE" library="HyTechDevices" deviceset="RESISTOR" device="0805-RES" value="3.3kΩ"/>
+<part name="DISCHARGE" library="HyTechDevices" deviceset="RESISTOR" device="PWR163" value="5Ω"/>
+<part name="PFET" library="HyTechDevices" deviceset="P-CHANNEL_MOSFET_DMP3099L-7" device=""/>
 <part name="R" library="HyTechDevices" deviceset="RESISTOR" device="0805-RES" value="100Ω"/>
 <part name="C" library="HyTechDevices" deviceset="CAP" device="0805" value="10nF"/>
@@
 </plain>
 <instances>
-<instance part="GATE1" gate="G$1" x="55.88" y="25.4"/>
-<instance part="W1" gate="G$1" x="35.56" y="12.7" rot="R270"/>
-<instance part="PFET1" gate="G$1" x="40.64" y="22.86" smashed="yes" rot="R180">
+<instance part="GATE" gate="G$1" x="55.88" y="25.4"/>
+<instance part="DISCHARGE" gate="G$1" x="35.56" y="12.7" rot="R270"/>
+<instance part="PFET" gate="G$1" x="40.64" y="22.86" smashed="yes" rot="R180">
 <attribute name="NAME" x="36.83" y="27.94" size="1.778" layer="95"/>
 </instance>
@@
 <wire x1="35.56" y1="43.18" x2="35.56" y2="25.4" width="0.1524" layer="91"/>
 <wire x1="35.56" y1="43.18" x2="27.94" y2="43.18" width="0.1524" layer="91"/>
-<pinref part="PFET1" gate="G$1" pin="S"/>
+<pinref part="PFET" gate="G$1" pin="S"/>
 <label x="27.94" y="43.18" size="1.778" layer="95" rot="R180" xref="yes"/>
 <pinref part="R" gate="G$1" pin="1"/>
@@
 <net name="GATE" class="0">
 <segment>
-<pinref part="GATE1" gate="G$1" pin="1"/>
+<pinref part="GATE" gate="G$1" pin="1"/>
 <wire x1="45.72" y1="25.4" x2="50.8" y2="25.4" width="0.1524" layer="91"/>
-<pinref part="PFET1" gate="G$1" pin="G"/>
+<pinref part="PFET" gate="G$1" pin="G"/>
 </segment>
 </net>
 <net name="S(N)" class="0">
 <segment>
-<pinref part="GATE1" gate="G$1" pin="2"/>
+<pinref part="GATE" gate="G$1" pin="2"/>
 <wire x1="60.96" y1="25.4" x2="78.74" y2="25.4" width="0.1524" layer="91"/>
 <label x="78.74" y="25.4" size="1.778" layer="95" xref="yes"/>
@@
 <wire x1="35.56" y1="5.08" x2="27.94" y2="5.08" width="0.1524" layer="91"/>
 <label x="27.94" y="5.08" size="1.778" layer="95" rot="R180" xref="yes"/>
-<pinref part="W1" gate="G$1" pin="2"/>
+<pinref part="DISCHARGE" gate="G$1" pin="2"/>
 <wire x1="35.56" y1="7.62" x2="35.56" y2="5.08" width="0.1524" layer="91"/>
 </segment>
@@
 <net name="N$1" class="0">
 <segment>
-<pinref part="PFET1" gate="G$1" pin="D"/>
-<pinref part="W1" gate="G$1" pin="1"/>
+<pinref part="PFET" gate="G$1" pin="D"/>
+<pinref part="DISCHARGE" gate="G$1" pin="1"/>
 <wire x1="35.56" y1="20.32" x2="35.56" y2="17.78" width="0.1524" layer="91"/>
 </segment>
@@
 <parts>
 <part name="R1" library="HyTechDevices" deviceset="RESISTOR" device="0805-RES" value="10kΩ"/>
-<part name="R2" library="HyTechDevices" deviceset="RESISTOR" device="0805-RES" value="100Ω"/>
-<part name="C1" library="HyTechDevices" deviceset="CAP" device="0805" value="10nF"/>
+<part name="R" library="HyTechDevices" deviceset="RESISTOR" device="0805-RES" value="100Ω"/>
+<part name="C" library="HyTechDevices" deviceset="CAP" device="0805" value="10nF"/>
 <part name="SUPPLY27" library="supply2" deviceset="V-" device=""/>
 </parts>
@@
 <instances>
 <instance part="R1" gate="G$1" x="10.16" y="10.16" rot="R270"/>
-<instance part="R2" gate="G$1" x="0" y="0"/>
-<instance part="C1" gate="G$1" x="-10.16" y="-7.62"/>
+<instance part="R" gate="G$1" x="0" y="0"/>
+<instance part="C" gate="G$1" x="-10.16" y="-7.62"/>
 <instance part="SUPPLY27" gate="1" x="-10.16" y="-15.24"/>
 </instances>
@@
 <pinref part="R1" gate="G$1" pin="2"/>
 <wire x1="10.16" y1="-7.62" x2="10.16" y2="0" width="0.1524" layer="91"/>
-<pinref part="R2" gate="G$1" pin="2"/>
+<pinref part="R" gate="G$1" pin="2"/>
 <wire x1="10.16" y1="0" x2="10.16" y2="5.08" width="0.1524" layer="91"/>
 <wire x1="5.08" y1="0" x2="10.16" y2="0" width="0.1524" layer="91"/>
@@
 <net name="GPIO" class="0">
 <segment>
-<pinref part="R2" gate="G$1" pin="1"/>
-<pinref part="C1" gate="G$1" pin="1"/>
+<pinref part="R" gate="G$1" pin="1"/>
+<pinref part="C" gate="G$1" pin="1"/>
 <wire x1="-10.16" y1="-2.54" x2="-10.16" y2="0" width="0.1524" layer="91"/>
 <wire x1="-10.16" y1="0" x2="-5.08" y2="0" width="0.1524" layer="91"/>
@@
 <segment>
 <pinref part="SUPPLY27" gate="1" pin="V-"/>
-<pinref part="C1" gate="G$1" pin="2"/>
+<pinref part="C" gate="G$1" pin="2"/>
 <wire x1="-10.16" y1="-12.7" x2="-10.16" y2="-10.16" width="0.1524" layer="91"/>
 </segment>
@@
 <text x="-248.92" y="132.08" size="3.81" layer="97" align="bottom-right">CELL 9 IS SHARED BY
 CIRCUIT A AND CIRCUIT B</text>
+<text x="17.78" y="193.04" size="1.778" layer="95">ADP2360</text>
+<text x="17.78" y="-45.72" size="1.778" layer="95">ADP2360</text>
+<text x="60.96" y="68.58" size="1.778" layer="95">0Ω jumper resistors
+to set chip address</text>
+<text x="60.96" y="307.34" size="1.778" layer="95">0Ω jumper resistors
+to set chip address</text>
+<text x="0" y="302.26" size="1.778" layer="95">LTC6804-2</text>
+<text x="0" y="63.5" size="1.778" layer="95">LTC6804-2</text>
 </plain>
 <moduleinsts>
@@
 </segment>
 </net>
-<net name="GPIO1A" class="0">
-<segment>
-<portref moduleinst="THERM_FILTER6" port="GPIO"/>
-<wire x1="107.95" y1="297.18" x2="106.68" y2="297.18" width="0.1524" layer="91"/>
-<label x="106.68" y="297.18" size="1.778" layer="95" rot="R180" xref="yes"/>
-</segment>
-</net>
 <net name="IP_A" class="0">
 <segment>
@@
 <label x="20.32" y="246.38" size="1.778" layer="95" xref="yes"/>
 </segment>
+<segment>
+<portref moduleinst="THERM_FILTER6" port="GPIO"/>
+<wire x1="107.95" y1="297.18" x2="106.68" y2="297.18" width="0.1524" layer="91"/>
+<label x="106.68" y="297.18" size="1.778" layer="95" rot="R180" xref="yes"/>
+</segment>
 </net>
