File: Board Designs/Latch Manager/latch_THT.brd (EAGLE design)
At the start: 81.3 x 56.2 mm, 19 parts, among them IC1 SN74AHC00, IC2 SN74AHC74, IC3 SN74AHC00, IC4 SN74AHC74, IC6 SN74AHC00, U1 SA555P, X1 CONNECTOR-4, X2 CONNECTOR-2

Commit message: Keeping a single copy of latching board until one works and can be revised. Removed first attempts.
Changed lines of the file:
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@@
 <contactref element="IC6" pad="2"/>
 <wire x1="26.035" y1="49.911" x2="28.575" y2="49.911" width="0.6096" layer="16"/>
-<wire x1="46.99" y1="49.911" x2="46.99" y2="47.498" width="0.6096" layer="16"/>
-<wire x1="46.99" y1="47.498" x2="28.575" y2="47.498" width="0.6096" layer="16"/>
-<wire x1="28.575" y1="47.498" x2="28.575" y2="49.911" width="0.6096" layer="16"/>
+<wire x1="46.99" y1="47.498" x2="46.99" y2="49.911" width="0.6096" layer="16"/>
+<wire x1="28.575" y1="49.911" x2="28.575" y2="47.498" width="0.6096" layer="16"/>
 <via x="8.763" y="15.494" extent="1-16" drill="0.35"/>
 <wire x1="20.233" y1="15.494" x2="8.763" y2="15.494" width="0.6096" layer="16"/>
@@
 <wire x1="8.763" y1="15.494" x2="7.493" y2="16.764" width="0.6096" layer="1"/>
 <wire x1="7.493" y1="16.764" x2="7.493" y2="22.019" width="0.6096" layer="1"/>
+<wire x1="28.575" y1="47.498" x2="46.99" y2="47.498" width="0.6096" layer="16"/>
 </signal>
 <signal name="12V">
