File: Board Designs/BMS/BMS Microcontroller/BMS Microcontroller rev2.brd (EAGLE design)
At the start: 54.4 x 60.6 mm, 35 parts, among them X1 CONNECTOR-4, X2 RJ45-6L21-B, X3 CONNECTOR-4

Commit message: Updated resistor value, other values in BMS microcontroller and HV board, Update FSAE board rev2, restore FSAE board
Parts:
- R13: value 68 -> 430
Changed lines of the file:
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@@
 <?xml version="1.0" encoding="utf-8"?>
 <!DOCTYPE eagle SYSTEM "eagle.dtd">
-<eagle version="8.2.1">
+<eagle version="8.4.1">
 <drawing>
 <settings>
 <setting alwaysvectorfont="no"/>
+<setting keepoldvectorfont="yes"/>
 <setting verticaltext="up"/>
 </settings>
@@
 <param name="dpMaxLengthDifference" value="10mm"/>
 <param name="dpGapFactor" value="2.5"/>
-<param name="checkGrid" value="0"/>
 <param name="checkAngle" value="0"/>
 <param name="checkFont" value="1"/>
 <param name="checkRestrict" value="1"/>
+<param name="checkStop" value="0"/>
 <param name="useDiameter" value="13"/>
 <param name="maxErrors" value="50"/>
@@
 <element name="R11" library="HyTechDevices" package="0805" value="1k" x="13.2842" y="5.969" rot="MR90"/>
 <element name="R12" library="HyTechDevices" package="0805" value="2k" x="6.6802" y="27.559" rot="R270"/>
-<element name="R13" library="HyTechDevices" package="0805" value="68" x="4.3942" y="35.179"/>
+<element name="R13" library="HyTechDevices" package="0805" value="430" x="4.3942" y="35.179"/>
 <element name="R2" library="HyTechDevices" package="0805" value="100" x="14.0462" y="15.113" rot="MR180"/>
 <element name="R3" library="HyTechDevices" package="0805" value="100" x="9.7282" y="17.399" rot="MR180"/>
@@
 <compatibility>
 <note version="8.2" severity="warning">
-Since Version 8.2, Eagle supports online libraries. The ids
+Since Version 8.2, EAGLE supports online libraries. The ids
 of those online libraries will not be understood (or retained)
 with this version.
