File: Board Designs/Precharger Board/precharger_rev1.sch (EAGLE design)
At the start: 14 parts, among them IC1 SN74AHC74, K1 RELAY

Commit message: Revised precharger schematic
Parts:
- added R2: (no value), HyTechDevices:RESISTOR0805-RES
Connections:
- new net N$5: IC1B.CLK
- new net N$8: C3.2, R2.2
- net GND: now also R2.1; no longer C3.2, IC1B.CLK
Other:
- moved on the sheet: C3
Changed lines of the file:
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@@
 <part name="C3" library="HyTechDevices" deviceset="CAP" device="0805"/>
 <part name="GND7" library="HyTechSymbols" deviceset="GND" device=""/>
+<part name="R2" library="HyTechDevices" deviceset="RESISTOR" device="0805-RES"/>
 </parts>
 <sheets>
@@
 <wire x1="132.08" y1="-5.08" x2="63.5" y2="-5.08" width="0.1524" layer="103"/>
 <text x="63.5" y="-2.54" size="1.778" layer="91">battery_circuit</text>
-<wire x1="86.36" y1="96.52" x2="86.36" y2="12.7" width="0.1524" layer="103"/>
-<wire x1="86.36" y1="12.7" x2="243.84" y2="12.7" width="0.1524" layer="103"/>
-<wire x1="243.84" y1="12.7" x2="243.84" y2="96.52" width="0.1524" layer="103"/>
+<wire x1="86.36" y1="96.52" x2="86.36" y2="0" width="0.1524" layer="103"/>
+<wire x1="86.36" y1="0" x2="243.84" y2="0" width="0.1524" layer="103"/>
+<wire x1="243.84" y1="0" x2="243.84" y2="96.52" width="0.1524" layer="103"/>
 <wire x1="243.84" y1="96.52" x2="86.36" y2="96.52" width="0.1524" layer="103"/>
 </plain>
@@
 <instance part="SUPPLY2" gate="G$1" x="180.34" y="43.18"/>
 <instance part="SUPPLY3" gate="G$1" x="182.88" y="27.94"/>
-<instance part="C3" gate="G$1" x="182.88" y="22.86"/>
-<instance part="GND7" gate="1" x="182.88" y="17.78"/>
+<instance part="C3" gate="G$1" x="182.88" y="20.32"/>
+<instance part="GND7" gate="1" x="182.88" y="5.08"/>
+<instance part="R2" gate="G$1" x="182.88" y="12.7" rot="R90"/>
 </instances>
 <busses>
@@
 </segment>
 <segment>
-<pinref part="C3" gate="G$1" pin="2"/>
+<pinref part="R2" gate="G$1" pin="1"/>
 <pinref part="GND7" gate="1" pin="GND"/>
-<pinref part="IC1" gate="B" pin="CLK"/>
-<wire x1="172.72" y1="40.64" x2="177.8" y2="40.64" width="0.1524" layer="91"/>
-<wire x1="177.8" y1="40.64" x2="177.8" y2="20.32" width="0.1524" layer="91"/>
-<wire x1="177.8" y1="20.32" x2="182.88" y2="20.32" width="0.1524" layer="91"/>
-<junction x="182.88" y="20.32"/>
 </segment>
 </net>
@@
 <pinref part="SUPPLY3" gate="G$1" pin="VIN"/>
 <pinref part="C3" gate="G$1" pin="1"/>
+<wire x1="182.88" y1="25.4" x2="182.88" y2="27.94" width="0.1524" layer="91"/>
 </segment>
 </net>
@@
 </segment>
 </net>
+<net name="N$5" class="0">
+<segment>
+<pinref part="IC1" gate="B" pin="CLK"/>
+<wire x1="172.72" y1="40.64" x2="177.8" y2="40.64" width="0.1524" layer="91"/>
+</segment>
+</net>
+<net name="N$8" class="0">
+<segment>
+<pinref part="C3" gate="G$1" pin="2"/>
+<pinref part="R2" gate="G$1" pin="2"/>
+</segment>
+</net>

Commit message: Revised some stuff
Parts:
- added R3, R4, R5, R6: (no value), HyTechDevices:RESISTOR0805-RES
- added U$4: MCP6542PDIP, HyTechDevices:MCP6542PDIP
Connections:
- new net N$10: R4.1, R5.2, U$4.VINA-
- new net N$9: R6.2, U$1.BASE
- net GND: now also C3.2, R5.1, U$4.VSS
- net N$5: now also U$4.VOUTA
- net N$7: now also R6.1; no longer U$1.BASE
- net N$8: now also C3.1, R3.1, U$4.VINA+; no longer C3.2
- net VIN: now also R3.2, R4.2, U$4.VDD; no longer C3.1
Other:
- note added: "r2/(r3+r4) > r5/(r4+r5)"
- moved on the sheet: C3, Q1, R2
Changed lines of the file:
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@@
 <part name="GND7" library="HyTechSymbols" deviceset="GND" device=""/>
 <part name="R2" library="HyTechDevices" deviceset="RESISTOR" device="0805-RES"/>
+<part name="R3" library="HyTechDevices" deviceset="RESISTOR" device="0805-RES"/>
+<part name="U$4" library="HyTechDevices" deviceset="MCP6542" device="PDIP"/>
+<part name="SUPPLY5" library="HyTechSymbols" deviceset="VIN" device=""/>
+<part name="R4" library="HyTechDevices" deviceset="RESISTOR" device="0805-RES"/>
+<part name="R5" library="HyTechDevices" deviceset="RESISTOR" device="0805-RES"/>
+<part name="GND8" library="HyTechSymbols" deviceset="GND" device=""/>
+<part name="GND9" library="HyTechSymbols" deviceset="GND" device=""/>
+<part name="SUPPLY6" library="HyTechSymbols" deviceset="VIN" device=""/>
+<part name="R6" library="HyTechDevices" deviceset="RESISTOR" device="0805-RES"/>
 </parts>
 <sheets>
@@
 <wire x1="243.84" y1="0" x2="243.84" y2="96.52" width="0.1524" layer="103"/>
 <wire x1="243.84" y1="96.52" x2="86.36" y2="96.52" width="0.1524" layer="103"/>
+<text x="203.2" y="5.08" size="1.778" layer="91">r2/(r3+r4) &gt; r5/(r4+r5)</text>
 </plain>
 <instances>
@@
 <instance part="GND3" gate="1" x="109.22" y="-15.24"/>
 <instance part="C2" gate="G$1" x="198.12" y="81.28"/>
-<instance part="Q1" gate="G$1" x="218.44" y="76.2"/>
-<instance part="SUPPLY4" gate="G$1" x="220.98" y="88.9"/>
+<instance part="Q1" gate="G$1" x="256.54" y="76.2"/>
+<instance part="SUPPLY4" gate="G$1" x="259.08" y="88.9"/>
 <instance part="GND1" gate="1" x="187.96" y="88.9" rot="R180"/>
 <instance part="GND2" gate="1" x="198.12" y="88.9" rot="R180"/>
@@
 <instance part="SUPPLY2" gate="G$1" x="180.34" y="43.18"/>
 <instance part="SUPPLY3" gate="G$1" x="182.88" y="27.94"/>
-<instance part="C3" gate="G$1" x="182.88" y="20.32"/>
+<instance part="C3" gate="G$1" x="182.88" y="12.7"/>
 <instance part="GND7" gate="1" x="182.88" y="5.08"/>
-<instance part="R2" gate="G$1" x="182.88" y="12.7" rot="R90"/>
+<instance part="R2" gate="G$1" x="190.5" y="12.7" rot="R90"/>
+<instance part="R3" gate="G$1" x="182.88" y="22.86" rot="R90"/>
+<instance part="U$4" gate="G$1" x="205.74" y="22.86"/>
+<instance part="SUPPLY5" gate="G$1" x="228.6" y="43.18"/>
+<instance part="R4" gate="G$1" x="228.6" y="38.1" rot="R90"/>
+<instance part="R5" gate="G$1" x="228.6" y="27.94" rot="R90"/>
+<instance part="GND8" gate="1" x="228.6" y="20.32"/>
+<instance part="GND9" gate="1" x="203.2" y="12.7"/>
+<instance part="SUPPLY6" gate="G$1" x="220.98" y="22.86"/>
+<instance part="R6" gate="G$1" x="165.1" y="53.34"/>
 </instances>
 <busses>
@@
 <segment>
 <pinref part="POWER_RES" gate="G$1" pin="1"/>
-<wire x1="91.44" y1="38.1" x2="96.52" y2="38.1" width="0.1524" layer="91"/>
+<wire x1="73.66" y1="38.1" x2="96.52" y2="38.1" width="0.1524" layer="91"/>
 <wire x1="96.52" y1="38.1" x2="96.52" y2="43.18" width="0.1524" layer="91"/>
 <wire x1="96.52" y1="38.1" x2="121.92" y2="38.1" width="0.1524" layer="91"/>
@@
 <pinref part="U$3" gate="G$1" pin="GND1"/>
 <wire x1="121.92" y1="76.2" x2="154.94" y2="76.2" width="0.1524" layer="91"/>
-<label x="91.44" y="38.1" size="1.27" layer="95" rot="R180" xref="yes"/>
+<label x="73.66" y="38.1" size="1.27" layer="95" rot="R180" xref="yes"/>
 </segment>
 <segment>
@@
 <wire x1="96.52" y1="68.58" x2="96.52" y2="78.74" width="0.1524" layer="91"/>
 <pinref part="LED_RES" gate="G$1" pin="1"/>
-<wire x1="96.52" y1="78.74" x2="91.44" y2="78.74" width="0.1524" layer="91"/>
+<wire x1="96.52" y1="78.74" x2="73.66" y2="78.74" width="0.1524" layer="91"/>
 <wire x1="96.52" y1="78.74" x2="106.68" y2="78.74" width="0.1524" layer="91"/>
 <junction x="96.52" y="78.74"/>
-<label x="91.44" y="78.74" size="1.27" layer="95" rot="R180" xref="yes"/>
+<label x="73.66" y="78.74" size="1.27" layer="95" rot="R180" xref="yes"/>
 </segment>
 <segment>
@@
 </segment>
 <segment>
+<pinref part="C3" gate="G$1" pin="2"/>
+<pinref part="GND7" gate="1" pin="GND"/>
 <pinref part="R2" gate="G$1" pin="1"/>
-<pinref part="GND7" gate="1" pin="GND"/>
+<wire x1="190.5" y1="7.62" x2="182.88" y2="7.62" width="0.1524" layer="91"/>
+<junction x="182.88" y="7.62"/>
+<wire x1="182.88" y1="7.62" x2="182.88" y2="10.16" width="0.1524" layer="91"/>
+</segment>
+<segment>
+<pinref part="R5" gate="G$1" pin="1"/>
+<pinref part="GND8" gate="1" pin="GND"/>
+</segment>
+<segment>
+<pinref part="U$4" gate="G$1" pin="VSS"/>
+<pinref part="GND9" gate="1" pin="GND"/>
 </segment>
 </net>
@@
 <wire x1="198.12" y1="76.2" x2="203.2" y2="76.2" width="0.1524" layer="91"/>
 <pinref part="Q1" gate="G$1" pin="BASE"/>
-<wire x1="203.2" y1="76.2" x2="215.9" y2="76.2" width="0.1524" layer="91"/>
+<wire x1="203.2" y1="76.2" x2="254" y2="76.2" width="0.1524" layer="91"/>
 <wire x1="203.2" y1="76.2" x2="203.2" y2="45.72" width="0.1524" layer="91"/>
 <junction x="203.2" y="76.2"/>
@@
 <segment>
 <pinref part="Q1" gate="G$1" pin="EMITTER"/>
-<wire x1="220.98" y1="71.12" x2="220.98" y2="58.42" width="0.1524" layer="91"/>
-<wire x1="220.98" y1="58.42" x2="223.52" y2="58.42" width="0.1524" layer="91"/>
-<label x="223.52" y="58.42" size="1.27" layer="95" xref="yes"/>
+<wire x1="259.08" y1="71.12" x2="259.08" y2="58.42" width="0.1524" layer="91"/>
+<wire x1="259.08" y1="58.42" x2="261.62" y2="58.42" width="0.1524" layer="91"/>
+<label x="261.62" y="58.42" size="1.27" layer="95" xref="yes"/>
 </segment>
 </net>
@@
 <pinref part="Q1" gate="G$1" pin="COLLECTOR"/>
 <pinref part="SUPPLY4" gate="G$1" pin="VIN"/>
-<wire x1="220.98" y1="81.28" x2="220.98" y2="88.9" width="0.1524" layer="91"/>
+<wire x1="259.08" y1="81.28" x2="259.08" y2="88.9" width="0.1524" layer="91"/>
 </segment>
 </net>
@@
 <segment>
 <pinref part="SUPPLY3" gate="G$1" pin="VIN"/>
-<pinref part="C3" gate="G$1" pin="1"/>
-<wire x1="182.88" y1="25.4" x2="182.88" y2="27.94" width="0.1524" layer="91"/>
+<pinref part="R3" gate="G$1" pin="2"/>
+</segment>
+<segment>
+<pinref part="SUPPLY5" gate="G$1" pin="VIN"/>
+<pinref part="R4" gate="G$1" pin="2"/>
+</segment>
+<segment>
+<pinref part="U$4" gate="G$1" pin="VDD"/>
+<pinref part="SUPPLY6" gate="G$1" pin="VIN"/>
 </segment>
 </net>
@@
 <wire x1="147.32" y1="35.56" x2="144.78" y2="35.56" width="0.1524" layer="91"/>
 <wire x1="144.78" y1="35.56" x2="144.78" y2="53.34" width="0.1524" layer="91"/>
-<wire x1="144.78" y1="53.34" x2="187.96" y2="53.34" width="0.1524" layer="91"/>
+<wire x1="144.78" y1="53.34" x2="160.02" y2="53.34" width="0.1524" layer="91"/>
+<pinref part="R6" gate="G$1" pin="1"/>
+</segment>
+</net>
+<net name="N$5" class="0">
+<segment>
+<pinref part="U$4" gate="G$1" pin="VOUTA"/>
+<wire x1="203.2" y1="22.86" x2="187.96" y2="22.86" width="0.1524" layer="91"/>
+<wire x1="187.96" y1="22.86" x2="187.96" y2="38.1" width="0.1524" layer="91"/>
+<wire x1="187.96" y1="38.1" x2="172.72" y2="38.1" width="0.1524" layer="91"/>
+<pinref part="IC1" gate="B" pin="CLK"/>
+<wire x1="172.72" y1="38.1" x2="172.72" y2="40.64" width="0.1524" layer="91"/>
+</segment>
+</net>
+<net name="N$8" class="0">
+<segment>
+<pinref part="C3" gate="G$1" pin="1"/>
+<pinref part="R3" gate="G$1" pin="1"/>
+<pinref part="R2" gate="G$1" pin="2"/>
+<wire x1="190.5" y1="17.78" x2="182.88" y2="17.78" width="0.1524" layer="91"/>
+<junction x="182.88" y="17.78"/>
+<pinref part="U$4" gate="G$1" pin="VINA+"/>
+<wire x1="190.5" y1="17.78" x2="203.2" y2="17.78" width="0.1524" layer="91"/>
+<junction x="190.5" y="17.78"/>
+</segment>
+</net>
+<net name="N$10" class="0">
+<segment>
+<pinref part="U$4" gate="G$1" pin="VINA-"/>
+<wire x1="203.2" y1="20.32" x2="200.66" y2="20.32" width="0.1524" layer="91"/>
+<wire x1="200.66" y1="20.32" x2="200.66" y2="33.02" width="0.1524" layer="91"/>
+<pinref part="R4" gate="G$1" pin="1"/>
+<pinref part="R5" gate="G$1" pin="2"/>
+<wire x1="200.66" y1="33.02" x2="228.6" y2="33.02" width="0.1524" layer="91"/>
+<junction x="228.6" y="33.02"/>
+</segment>
+</net>
+<net name="N$9" class="0">
+<segment>
 <pinref part="U$1" gate="G$1" pin="BASE"/>
+<pinref part="R6" gate="G$1" pin="2"/>
+<wire x1="170.18" y1="53.34" x2="187.96" y2="53.34" width="0.1524" layer="91"/>
 <wire x1="187.96" y1="53.34" x2="187.96" y2="68.58" width="0.1524" layer="91"/>
 </segment>
 </net>
-<net name="N$5" class="0">
-<segment>
-<pinref part="IC1" gate="B" pin="CLK"/>
-<wire x1="172.72" y1="40.64" x2="177.8" y2="40.64" width="0.1524" layer="91"/>
-</segment>
-</net>
-<net name="N$8" class="0">
-<segment>
-<pinref part="C3" gate="G$1" pin="2"/>
-<pinref part="R2" gate="G$1" pin="2"/>
-</segment>
-</net>

Commit message: Revised precharger schematic
Parts:
- removed U$1: =, HyTechDevices:NPN_BCP56T1
- removed U$4: MCP6542PDIP, HyTechDevices:MCP6542PDIP
- added LED1: (no value), HyTechDevices:LED-0805
- added R7, R8, R9: (no value), HyTechDevices:RESISTOR0805-RES
Connections:
- removed net N$1: C2.2, R1.2, U$1.COLLECTOR, U$3.EM1
- new net N$11: R7.1, R8.2, U$2.VINA-
- new net N$12: LED1.A, R9.1
- net GND: now also LED1.C, R8.1, U$3.EM2, U$3.GND2; no longer U$1.EMITTER, U$2.VINA-, U$4.VSS
- net N$10: now also U$2.VINB-; no longer U$4.VINA-
- net N$5: now also U$2.VOUTB; no longer U$4.VOUTA
- net N$7: now also R9.2
- net N$8: now also U$2.VINB+; no longer U$4.VINA+
- net N$9: no longer U$1.BASE
- net RELAY: now also C2.2, R1.2, U$3.C2, U$3.EM1
- net VIN: now also R7.2; no longer U$4.VDD
Other:
- note added: "configure so v = ~0.3V"
- moved on the sheet: R1, R6

Commit message: Revised precharger
Parts:
- added U$1: SOLID_STATE_RELAY_G3VM-41AY, HyTechDevices:SOLID_STATE_RELAY_G3VM-41AY
Connections:
- new net N$1: POWER_RES2.2, U$1.IO2
- net A: now also U$1.IO1; no longer POWER_RES2.2
- net GND: now also U$1.LED-
- net VIN: now also U$1.LED+
Changed lines of the file:
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@@
 <part name="R9" library="HyTechDevices" deviceset="RESISTOR" device="0805-RES"/>
 <part name="LED1" library="HyTechDevices" deviceset="LED" device="-0805"/>
+<part name="U$1" library="HyTechDevices" deviceset="SOLID_STATE_RELAY" device="_G3VM-41AY" value=""/>
+<part name="SUPPLY7" library="HyTechSymbols" deviceset="VIN" device=""/>
+<part name="GND11" library="HyTechSymbols" deviceset="GND" device=""/>
 </parts>
 <sheets>
@@
 <instance part="R9" gate="G$1" x="144.78" y="30.48" rot="R90"/>
 <instance part="LED1" gate="LED" x="144.78" y="22.86"/>
+<instance part="U$1" gate="G$1" x="114.3" y="60.96" rot="MR0"/>
+<instance part="SUPPLY7" gate="G$1" x="124.46" y="66.04"/>
+<instance part="GND11" gate="1" x="124.46" y="53.34"/>
 </instances>
 <busses>
@@
 <wire x1="73.66" y1="38.1" x2="96.52" y2="38.1" width="0.1524" layer="91"/>
 <wire x1="96.52" y1="38.1" x2="96.52" y2="43.18" width="0.1524" layer="91"/>
-<wire x1="96.52" y1="38.1" x2="121.92" y2="38.1" width="0.1524" layer="91"/>
-<wire x1="121.92" y1="38.1" x2="121.92" y2="76.2" width="0.1524" layer="91"/>
+<wire x1="96.52" y1="38.1" x2="129.54" y2="38.1" width="0.1524" layer="91"/>
+<wire x1="129.54" y1="38.1" x2="129.54" y2="76.2" width="0.1524" layer="91"/>
 <junction x="96.52" y="38.1"/>
 <pinref part="U$3" gate="G$1" pin="GND1"/>
-<wire x1="121.92" y1="76.2" x2="154.94" y2="76.2" width="0.1524" layer="91"/>
+<wire x1="129.54" y1="76.2" x2="154.94" y2="76.2" width="0.1524" layer="91"/>
 <label x="73.66" y="38.1" size="1.27" layer="95" rot="R180" xref="yes"/>
 </segment>
@@
 <net name="A" class="0">
 <segment>
-<pinref part="POWER_RES2" gate="G$1" pin="2"/>
-<wire x1="96.52" y1="68.58" x2="96.52" y2="78.74" width="0.1524" layer="91"/>
 <pinref part="LED_RES" gate="G$1" pin="1"/>
+<wire x1="106.68" y1="78.74" x2="96.52" y2="78.74" width="0.1524" layer="91"/>
+<label x="73.66" y="78.74" size="1.27" layer="95" rot="R180" xref="yes"/>
 <wire x1="96.52" y1="78.74" x2="73.66" y2="78.74" width="0.1524" layer="91"/>
-<wire x1="96.52" y1="78.74" x2="106.68" y2="78.74" width="0.1524" layer="91"/>
+<wire x1="104.14" y1="73.66" x2="96.52" y2="73.66" width="0.1524" layer="91"/>
+<wire x1="96.52" y1="73.66" x2="96.52" y2="78.74" width="0.1524" layer="91"/>
 <junction x="96.52" y="78.74"/>
-<label x="73.66" y="78.74" size="1.27" layer="95" rot="R180" xref="yes"/>
+<pinref part="U$1" gate="G$1" pin="IO1"/>
+<wire x1="104.14" y1="73.66" x2="104.14" y2="63.5" width="0.1524" layer="91"/>
 </segment>
 <segment>
@@
 <pinref part="GND10" gate="1" pin="GND"/>
 <pinref part="LED1" gate="LED" pin="C"/>
+</segment>
+<segment>
+<pinref part="U$1" gate="G$1" pin="LED-"/>
+<pinref part="GND11" gate="1" pin="GND"/>
+<wire x1="124.46" y1="58.42" x2="124.46" y2="55.88" width="0.1524" layer="91"/>
 </segment>
 </net>
@@
 <pinref part="SUPPLY6" gate="G$1" pin="VIN"/>
 </segment>
+<segment>
+<pinref part="U$1" gate="G$1" pin="LED+"/>
+<pinref part="SUPPLY7" gate="G$1" pin="VIN"/>
+<wire x1="124.46" y1="63.5" x2="124.46" y2="66.04" width="0.1524" layer="91"/>
+</segment>
 </net>
 <net name="N$6" class="0">
@@
 </segment>
 </net>
+<net name="N$1" class="0">
+<segment>
+<pinref part="POWER_RES2" gate="G$1" pin="2"/>
+<wire x1="96.52" y1="68.58" x2="96.52" y2="71.12" width="0.1524" layer="91"/>
+<wire x1="96.52" y1="71.12" x2="101.6" y2="71.12" width="0.1524" layer="91"/>
+<pinref part="U$1" gate="G$1" pin="IO2"/>
+<wire x1="101.6" y1="71.12" x2="101.6" y2="58.42" width="0.1524" layer="91"/>
+<wire x1="101.6" y1="58.42" x2="104.14" y2="58.42" width="0.1524" layer="91"/>
+</segment>
+</net>
