File: Board Designs/Precharger Board/precharger_rev3.brd (EAGLE design)
At the start: 84.8 x 52.1 mm, 21 parts, among them X1 CONNECTOR-2, X2 CONNECTOR-2

Commit message: Precharger Board revision
Parts:
- removed R2: ~20ohm, HyTechDevices:AXIAL-0.3
- added X3: CONNECTOR-2, HyTechDevices:MINIFIT_5566-2
- added _: 22k, HyTechDevices:AXIAL-0.3
- C3: device HyTechDevices:CAP-PTH-5MM -> HyTechDevices:CAP-PTH-SMALL
- LED_RES: value ~670ohm -> 22k
- moved X1 2.84 mm to (72.4, 36.8)
Connections:
- removed net N$12: R2.P$2, U$1.3
- removed net N$3: C3.1, R3.P$1, R6.P$2, U$2.5
- new net N$7: C3.1, R3.P$1, R6.P$2, U$2.5, U$3.2
- net A1: now also _.P$1
- net GND: now also U$1.31, X3.2; no longer U$1.32
- net N$1: now also U$1.3; no longer R2.P$1
- net N$10: no longer U$3.2
- net N$4: now also _.P$2
- net NODE: now also U$1.32, X3.1; no longer U$1.31
Routing:
- net N$7: track 0.00 -> 62.9 mm, vias 0 -> 2
- net N$3: track 49.4 -> 0.00 mm, vias 1 -> 0
- net NODE: track 121.8 -> 161.9 mm, vias 0 -> 2
- net N$1: track 45.9 -> 69.6 mm
- net N$12: track 18.8 -> 0.00 mm
- net SIGNAL: track 50.9 -> 48.0 mm
- net N$10: track 53.2 -> 50.7 mm
- net A1: track 29.8 -> 32.4 mm
- net N$4: track 4.34 -> 6.35 mm
Other:
- board size 84.8 x 52.1 mm -> 86 x 52.1 mm
