File: Board Designs/External Boards/FH Charger Control Board/ShutdownOverview.sch (EAGLE design)
At the start: 41 parts, among them K1 RELAY, K2 RELAY, X2 CONNECTOR-12

Commit message: Fixed labelling for shutdown circuit overview for FH and FSAE ESFs
Parts:
- removed BMS_SSR1, IMD_SSR1, SOFT_SSR: CPC1002N, HyTechDevices:CPC1002N
- removed BRB, BRB1: SWITCH_SPST, HyTechSymbols:SWITCH_SPST
- removed D4, D5, D6: DIODE0805, HyTechDevices:DIODE0805
- removed K2: RELAY, HyTechSymbols:RELAY
- removed LED13, LED6, LED9: (no value), HyTechDevices:LED-0805
- removed R11, R15, R6: (no value), HyTechDevices:RESISTOR0805-RES
- removed S5, S6: (no value), HyTechDevices:BTN_10-XX
- removed U$6, U$7: G2RL-2-DC12, HyTechDevices:G2RL-2-DC12
- removed U$8: G5LE, HyTechDevices:G5LE
- removed X2: CONNECTOR-12, HyTechDevices:CONNECTOR-12
- added K3: RELAY, HyTechSymbols:RELAY
Connections:
- removed net +12V: BMS_SSR1.DC+, IMD_SSR1.DC+, SOFT_SSR.DC+
- removed net BMS: BMS_SSR1.CONTROL+
- removed net BMS_12V: BMS_SSR1.DC-, R11.2, S6.P, S6.P1, U$7.4, X2-8.S
- removed net BMS_OK: D5.C, S6.S, S6.S1, U$7.3, U$7.COIL-, X2-7.S
- removed net IMD: IMD_SSR1.CONTROL+
- removed net IMD_12V: IMD_SSR1.DC-, R6.2, S5.P, S5.P1, U$6.4, X2-2.S
- removed net IMD_OK: D4.C, S5.S, S5.S1, U$6.3, U$6.COIL-, X2-1.S
- removed net N$10: BRB.S
- removed net N$14: LED13.A, R15.1
- removed net N$2: U$7.5, U$8.P
- removed net N$28: BRB1.S
- removed net N$29: D6.C, U$8.COIL-
- removed net N$30: U$8.O
- removed net N$6: LED6.A, R6.1
- removed net N$7: LED9.A, R11.1
- removed net SW_KILL: SOFT_SSR.CONTROL+
- removed net SW_KILL_RELAY: D6.A, R15.2, SOFT_SSR.DC-, U$8.COIL+
- new net +5V: K3.P
- net GND: now also K3.1; no longer BMS_SSR1.CONTROL-, D4.A, D5.A, IMD_SSR1.CONTROL-, LED13.C, LED6.C, LED9.C, SOFT_SSR.CONTROL-, U$6.COIL+, U$7.COIL+
- net N$1: now also K3.S; no longer U$6.5, U$7.6
- net SHUTDOWN_ENABLE: now also K3.2; no longer BRB.P
