File: Board Designs/HV Board/HV Board rev2.sch (EAGLE design)
At the start: 95 parts, among them IC2 NE5532SOIC, IC3 NE5532SOIC

Commit message: Tweaks to murata board
Parts:
- C1: value 220uF -> 180µF
Changed lines of the file:
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@@
 <?xml version="1.0" encoding="utf-8"?>
 <!DOCTYPE eagle SYSTEM "eagle.dtd">
-<eagle version="8.4.1">
+<eagle version="9.0.1">
 <drawing>
 <settings>
@@
 <part name="R9" library="HyTechDevices" deviceset="RESISTOR" device="0805-RES" value="8.2k"/>
 <part name="R8" library="HyTechDevices" deviceset="RESISTOR" device="0805-RES" value="8.2k"/>
-<part name="C1" library="HyTechDevices" deviceset="CAP" device="" value="220uF"/>
+<part name="C1" library="HyTechDevices" deviceset="CAP" device="" value="180µF"/>
 <part name="U$3" library="HyTechDevices" deviceset="JUMPER" device=".3"/>
 <part name="U$4" library="HyTechDevices" deviceset="JUMPER" device=".3"/>
